File: design/thermistors/thermistors.kicad_pcb (KiCad board)
At the start: 2 copper layers, 76.2 x 35.6 mm, 21 parts, among them J1 Conn_01x02, J10 Conn_01x02, J2 Conn_01x08, J3 Conn_01x02, J4 Conn_01x02, J5 Conn_01x02, J6 Conn_01x02, J7 Conn_01x02, J8 Conn_01x02, J9 Conn_01x02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

Commit message: Reroute PCB and add schematic pdf.
Parts:
- added ?: MountingHole_3.2mm_M3_Pad, Mounting_Holes:MountingHole_3.2mm_M3_Pad, F.Cu at (201.3, 98.4)
- added ?: MountingHole_3.2mm_M3_Pad, Mounting_Holes:MountingHole_3.2mm_M3_Pad, F.Cu at (118.7, 125.1)
- added ?: MountingHole_3.2mm_M3_Pad, Mounting_Holes:MountingHole_3.2mm_M3_Pad, F.Cu at (201.3, 125.1)
- added REF**: MountingHole_3.2mm_M3_Pad, Mounting_Holes:MountingHole_3.2mm_M3_Pad, F.Cu at (118.7, 98.4)
Other:
- board size 76.2 x 35.6 mm -> 93 x 35.6 mm
Changed lines of the file:
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@@
     (links 38)
     (no_connects 0)
-    (area 122.445 94.105 196.585001 129.515)
+    (area 121.844999 93.904999 198.195001 129.615001)
     (thickness 1.6)
     (drawings 4)
     (tracks 98)
     (zones 0)
-    (modules 21)
+    (modules 25)
     (nets 12)
   )
@@
     (pad_to_mask_clearance 0.2)
     (aux_axis_origin 0 0)
-    (visible_elements FFFFFF7F)
+    (visible_elements FFFEFF7F)
     (pcbplotparams
       (layerselection 0x00030_80000001)
@@
     )
   )
-  (gr_line (start 121.92 129.54) (end 198.12 129.54) (angle 90) (layer Edge.Cuts) (width 0.15))
-  (gr_line (start 121.92 93.98) (end 121.92 129.54) (angle 90) (layer Edge.Cuts) (width 0.15))
-  (gr_line (start 198.12 93.98) (end 198.12 129.54) (angle 90) (layer Edge.Cuts) (width 0.15))
-  (gr_line (start 121.92 93.98) (end 198.12 93.98) (angle 90) (layer Edge.Cuts) (width 0.15))
+  (module Mounting_Holes:MountingHole_3.2mm_M3_Pad (layer F.Cu)
+    (at 118.745 98.425)
+    (descr "Mounting Hole 3.2mm, M3")
+    (tags "mounting hole 3.2mm m3")
+    (attr virtual)
+    (fp_text reference REF** (at 0 -4.2) (layer F.SilkS) hide
+      (effects (font (size 1 1) (thickness 0.15)))
+    )
+    (fp_text value MountingHole_3.2mm_M3_Pad (at 0 4.2) (layer F.Fab)
+      (effects (font (size 1 1) (thickness 0.15)))
+    )
+    (fp_text user %R (at 0.3 0) (layer F.Fab)
+      (effects (font (size 1 1) (thickness 0.15)))
+    )
+    (fp_circle (center 0 0) (end 3.2 0) (layer Cmts.User) (width 0.15))
+    (fp_circle (center 0 0) (end 3.45 0) (layer F.CrtYd) (width 0.05))
+    (pad 1 thru_hole circle (at 0 0) (size 6.4 6.4) (drill 3.2) (layers *.Cu *.Mask))
+  )
+  (module Mounting_Holes:MountingHole_3.2mm_M3_Pad (layer F.Cu)
+    (at 201.295 98.425)
+    (descr "Mounting Hole 3.2mm, M3")
+    (tags "mounting hole 3.2mm m3")
+    (attr virtual)
+    (fp_text reference "" (at 0 -4.2) (layer F.SilkS)
+      (effects (font (size 1 1) (thickness 0.15)))
+    )
+    (fp_text value MountingHole_3.2mm_M3_Pad (at 0 4.2) (layer F.Fab)
+      (effects (font (size 1 1) (thickness 0.15)))
+    )
+    (fp_text user %R (at 0.3 0) (layer F.Fab)
+      (effects (font (size 1 1) (thickness 0.15)))
+    )
+    (fp_circle (center 0 0) (end 3.2 0) (layer Cmts.User) (width 0.15))
+    (fp_circle (center 0 0) (end 3.45 0) (layer F.CrtYd) (width 0.05))
+    (pad 1 thru_hole circle (at 0 0) (size 6.4 6.4) (drill 3.2) (layers *.Cu *.Mask))
+  )
+  (module Mounting_Holes:MountingHole_3.2mm_M3_Pad (layer F.Cu)
+    (at 118.745 125.095)
+    (descr "Mounting Hole 3.2mm, M3")
+    (tags "mounting hole 3.2mm m3")
+    (attr virtual)
+    (fp_text reference "" (at 0 -4.2) (layer F.SilkS)
+      (effects (font (size 1 1) (thickness 0.15)))
+    )
+    (fp_text value MountingHole_3.2mm_M3_Pad (at 0 4.2) (layer F.Fab)
+      (effects (font (size 1 1) (thickness 0.15)))
+    )
+    (fp_text user %R (at 0.3 0) (layer F.Fab)
+      (effects (font (size 1 1) (thickness 0.15)))
+    )
+    (fp_circle (center 0 0) (end 3.2 0) (layer Cmts.User) (width 0.15))
+    (fp_circle (center 0 0) (end 3.45 0) (layer F.CrtYd) (width 0.05))
+    (pad 1 thru_hole circle (at 0 0) (size 6.4 6.4) (drill 3.2) (layers *.Cu *.Mask))
+  )
+  (module Mounting_Holes:MountingHole_3.2mm_M3_Pad (layer F.Cu)
+    (at 201.295 125.095)
+    (descr "Mounting Hole 3.2mm, M3")
+    (tags "mounting hole 3.2mm m3")
+    (attr virtual)
+    (fp_text reference "" (at 0 -4.2) (layer F.SilkS)
+      (effects (font (size 1 1) (thickness 0.15)))
+    )
+    (fp_text value MountingHole_3.2mm_M3_Pad (at 0 4.2) (layer F.Fab)
+      (effects (font (size 1 1) (thickness 0.15)))
+    )
+    (fp_text user %R (at 0.3 0) (layer F.Fab)
+      (effects (font (size 1 1) (thickness 0.15)))
+    )
+    (fp_circle (center 0 0) (end 3.2 0) (layer Cmts.User) (width 0.15))
+    (fp_circle (center 0 0) (end 3.45 0) (layer F.CrtYd) (width 0.05))
+    (pad 1 thru_hole circle (at 0 0) (size 6.4 6.4) (drill 3.2) (layers *.Cu *.Mask))
+  )
+  (gr_line (start 113.665 129.54) (end 206.375 129.54) (angle 90) (layer Edge.Cuts) (width 0.15))
+  (gr_line (start 113.665 93.98) (end 206.375 93.98) (angle 90) (layer Edge.Cuts) (width 0.15))
+  (gr_line (start 113.538 93.98) (end 113.538 129.54) (angle 90) (layer Edge.Cuts) (width 0.15))
+  (gr_line (start 206.502 93.98) (end 206.502 129.54) (angle 90) (layer Edge.Cuts) (width 0.15))
   (segment (start 139.7 100.33) (end 139.192 100.33) (width 0.25) (layer F.Cu) (net 1))
   (segment (start 139.192 100.33) (end 135.382 104.14) (width 0.25) (layer F.Cu) (net 1))
@@
   (segment (start 135.382 104.14) (end 142.24 104.14) (width 0.25) (layer F.Cu) (net 1))
   (segment (start 142.24 104.14) (end 146.05 100.33) (width 0.25) (layer F.Cu) (net 1))
-  (segment (start 152.4 106.68) (end 152.4 106.172) (width 0.25) (layer B.Cu) (net 3) (status C00000))
-  (segment (start 152.4 106.172) (end 153.416 105.156) (width 0.25) (layer B.Cu) (net 3) (status 400000))
+  (segment (start 152.4 106.68) (end 152.4 106.172) (width 0.25) (layer B.Cu) (net 3))
+  (segment (start 152.4 106.172) (end 153.416 105.156) (width 0.25) (layer B.Cu) (net 3))
   (segment (start 146.812 105.156) (end 153.416 105.156) (width 0.25) (layer B.Cu) (net 3))
   (segment (start 153.416 105.156) (end 154.94 105.156) (width 0.25) (layer B.Cu) (net 3))
@@
   (via (at 155.194 102.616) (size 0.6) (drill 0.4) (layers F.Cu B.Cu) (net 3))
   (segment (start 155.194 102.616) (end 152.908 100.33) (width 0.25) (layer F.Cu) (net 3))
-  (segment (start 152.908 100.33) (end 151.13 100.33) (width 0.25) (layer F.Cu) (net 3) (status 800000))
+  (segment (start 152.908 100.33) (end 151.13 100.33) (width 0.25) (layer F.Cu) (net 3))
   (segment (start 151.13 100.33) (end 157.48 100.33) (width 0.25) (layer F.Cu) (net 3))
   (segment (start 165.608 105.156) (end 157.734 105.156) (width 0.25) (layer B.Cu) (net 3))

Commit message: Add schematics and pcb files for thermistor board
Parts:
- added G***: LOGO, RLCS_footprints:rocketry_logo_small_noletters, F.Cu at (198.7, 110.6)
Routing:
- net /therm_7: track 38.4 -> 32.8 mm
- net /therm_1: track 64.1 -> 60.8 mm
- net /therm_8: track 31.5 -> 28.4 mm
- net /therm_5: track 46.4 -> 43.9 mm
- net /therm_2: track 60.6 -> 58.2 mm
- net /therm_6: track 40.1 -> 37.9 mm
- net /therm_4: track 49.6 -> 47.4 mm
- net /therm_3: track 55.1 -> 53.8 mm
Other:
- board size 93 x 35.6 mm -> 92.7 x 35.6 mm
- board text added: "GND"
- board text added: "J=σE"
- board text added: "PWR"
- board text added: "SIGNAL OUT"
- board text added: "THERM CONN"
