File: design/strain_gauges_rtr/instr_amp.sch (KiCad schematic (older format))
At the start: 5 parts, among them J4 Conn_01x04, U3 INA826

Commit message: Add components for I2C Pancake
Parts:
- C5: symbol device:C -> strain_gauges_rtr-rescue:C-device
- R6, R7: symbol device:R -> strain_gauges_rtr-rescue:R-device
- U3: symbol daq_components:INA826 -> strain_gauges_rtr-rescue:INA826-daq_components
Changed lines of the file:
@@
 EESchema Schematic File Version 4
-LIBS:strain_gauges_rtr-cache
-EELAYER 26 0
+EELAYER 30 0
 EELAYER END
 $Descr A4 11693 8268
@@
 $EndDescr
 $Comp
-L daq_components:INA826 U3
+L strain_gauges_rtr-rescue:INA826-daq_components U3
 U 1 1 5ACAFA52
 P 5900 4100
@@
 	5100 3350 4950 3350
 $Comp
-L device:R R6
+L strain_gauges_rtr-rescue:R-device R6
 U 1 1 5ACAFBC2
 P 5000 4100
@@
 	6450 3950 6350 3950
 $Comp
-L device:C C5
+L strain_gauges_rtr-rescue:C-device C5
 U 1 1 5ACAFF7B
 P 6600 3700
@@
 G = 1 + 49.4K/RG
 $Comp
-L device:R R7
+L strain_gauges_rtr-rescue:R-device R7
 U 1 1 5ACB2059
 P 6500 4150
