File: design/strain_gauges_rtr/strain_gauges_rtr.sch (KiCad schematic (older format))
At the start: 17 parts, among them J1 Conn_01x03, J2 Conn_01x03, J3 Conn_01x08, P1 CONN_01X02, Q1 2N3096, U1 TL780-15, U2 LT1460-10

Commit message: Add components for I2C Pancake
Parts:
- C1, C2, C3, C4: symbol device:C -> strain_gauges_rtr-rescue:C-device
- F1: symbol device:Fuse -> strain_gauges_rtr-rescue:Fuse-device
- Q1: symbol device:Q_PNP_EBC -> strain_gauges_rtr-rescue:Q_PNP_EBC-device
- R1, R2, R3, R4, R5: symbol device:R -> strain_gauges_rtr-rescue:R-device
- U1: symbol daq_components:TL780-15 -> strain_gauges_rtr-rescue:TL780-15-daq_components
- U2: symbol daq_components:LT1460-10 -> strain_gauges_rtr-rescue:LT1460-10-daq_components
Changed lines of the file:
@@
 EESchema Schematic File Version 4
-LIBS:strain_gauges_rtr-cache
-EELAYER 26 0
+EELAYER 30 0
 EELAYER END
 $Descr A4 11693 8268
@@
 $EndDescr
 $Comp
-L device:R R1
+L strain_gauges_rtr-rescue:R-device R1
 U 1 1 5ACADCA3
 P 2300 1550
@@
 $EndComp
 $Comp
-L device:C C4
+L strain_gauges_rtr-rescue:C-device C4
 U 1 1 5ACADCAA
 P 3250 2850
@@
 $EndComp
 $Comp
-L device:C C1
+L strain_gauges_rtr-rescue:C-device C1
 U 1 1 5ACADCB7
 P 4050 1600
@@
 $EndComp
 $Comp
-L daq_components:+16V #PWR05
+L strain_gauges_rtr-rescue:+16V-daq_components #PWR05
 U 1 1 5ACADCD7
 P 2750 1050
@@
 $EndComp
 $Comp
-L daq_components:LT1460-10 U2
+L strain_gauges_rtr-rescue:LT1460-10-daq_components U2
 U 1 1 5ACADCDD
 P 2300 2400
@@
 $EndComp
 $Comp
-L device:Q_PNP_EBC Q1
+L strain_gauges_rtr-rescue:Q_PNP_EBC-device Q1
 U 1 1 5ACADCE4
 P 3150 1850
@@
 1.5 W, 200 mA
 $Comp
-L daq_components:+16V #PWR06
+L strain_gauges_rtr-rescue:+16V-daq_components #PWR06
 U 1 1 5ACAE219
 P 5450 1100
@@
 $EndComp
 $Comp
-L device:C C2
+L strain_gauges_rtr-rescue:C-device C2
 U 1 1 5ACAE225
 P 5600 1600
@@
 $EndComp
 $Comp
-L device:C C3
+L strain_gauges_rtr-rescue:C-device C3
 U 1 1 5ACAE22C
 P 6800 1600
@@
 $EndComp
 $Comp
-L daq_components:TL780-15 U1
+L strain_gauges_rtr-rescue:TL780-15-daq_components U1
 U 1 1 5ACAE23F
 P 6100 1000
@@
 $EndComp
 $Comp
-L device:R R3
+L strain_gauges_rtr-rescue:R-device R3
 U 1 1 5ACAEDCA
 P 9050 5100
@@
 $EndComp
 $Comp
-L device:R R5
+L strain_gauges_rtr-rescue:R-device R5
 U 1 1 5ACAEDD1
 P 9050 5450
@@
 $EndComp
 $Comp
-L device:R R2
+L strain_gauges_rtr-rescue:R-device R2
 U 1 1 5ACAEDDE
 P 8550 5100
@@
 $EndComp
 $Comp
-L device:R R4
+L strain_gauges_rtr-rescue:R-device R4
 U 1 1 5ACAEDE5
 P 8550 5450
@@
 Connection ~ 2750 1250
 $Comp
-L device:Fuse F1
+L strain_gauges_rtr-rescue:Fuse-device F1
 U 1 1 5ACB8796
 P 1950 1250
