File: design/I2C_Pancake/i2c_pancake.kicad_pcb (KiCad board)
At the start: 4 copper layers, 74.9 x 45 mm, 60 parts, among them J1 Conn_01x05_Male, J2 Conn_01x05_Male, J3 Conn_01x05_Female, J4 Conn_01x03, J5 Conn_01x03, J6 Conn_01x04, J7 Conn_01x04, J8 Conn_01x04, SW1 SW_DIP_x04, U1 INA826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

Commit message: Fix routing for +5V trace
Parts:
- U4: value HTSOP-J8_ROM -> BDJ0FC0WEFJ-E2
Connections:
- R1 pad 1: +5V -> VDD
- U4 pad 5: +5V -> VDD
Routing:
- net +5V: track 123.5 -> 104.4 mm, vias 2 -> 1
- net VDD: track 84.9 -> 102.7 mm
- net +10V: track 30.4 -> 32.5 mm
- net GND: track 69.5 -> 71.5 mm

Commit message: Make some last-minute PCB updates
Parts:
- added TP6: TestPoint, custom:TestPoint, F.Cu at (149.1, 112.6)
Connections:
- J3 pad 4: +5V -> VDD
Routing:
- net VDD: track 102.7 -> 127.0 mm
- net +5V: track 104.4 -> 96.0 mm, vias 1 -> 0
- net /SCL: track 114.8 -> 109.5 mm
Other:
- board text added: "Zachary Teper Oct-15-2020"
- board text removed: "Zachary Teper Oct-11-2020"
Changed lines of the file:
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@@
     (thickness 1.6)
     (drawings 40)
-    (tracks 583)
+    (tracks 591)
     (zones 0)
-    (modules 60)
+    (modules 61)
     (nets 48)
   )
@@
     (add_net "Net-(C1-Pad1)")
   )
+  (module custom:TestPoint (layer F.Cu)
+    (at 149.0726 112.5954)
+    (fp_text reference TP6 (at 0.0762 0.968) (layer F.SilkS)
+      (effects (font (size 1 1) (thickness 0.15)))
+    )
+    (fp_text value TestPoint (at 0 -0.5) (layer F.Fab)
+      (effects (font (size 1 1) (thickness 0.15)))
+    )
+    (fp_circle (center 0 3) (end 1 3) (layer F.SilkS) (width 0.12))
+    (pad 1 thru_hole circle (at 0 3) (size 1.524 1.524) (drill 0.762) (layers *.Cu *.Mask)
+      (net 33 VDD))
+  )
   (module footprints:MountingHole_3.2mm_M3_Pad (layer F.Cu)
     (at 160.454 130.853)
@@
       (net 1 GND))
     (pad 4 smd rect (at 7.62 0 90) (size 1 2) (layers B.Cu B.Paste B.Mask)
-      (net 11 +5V))
+      (net 33 VDD))
     (pad 5 smd rect (at 10.16 0 90) (size 1 2) (layers B.Cu B.Paste B.Mask)
       (net 19 /~MCLR))
@@
   (gr_line (start 93.854 134.253) (end 93.854 89.153) (layer Dwgs.User) (width 0.15))
   (gr_line (start 89.662 134.239) (end 164.554 134.239) (angle 90) (layer Edge.Cuts) (width 0.15))
-  (gr_text "Zachary Teper\nOct-11-2020" (at 157.354 105.153 90) (layer F.SilkS)
+  (gr_text "Zachary Teper\nOct-15-2020" (at 157.354 105.153 90) (layer F.SilkS)
     (effects (font (size 0.8 0.8) (thickness 0.12)) (justify left))
   )
@@
   (segment (start 153.147444 98.5266) (end 151.774424 99.89962) (width 0.3048) (layer F.Cu) (net 11))
   (segment (start 157.607 98.5266) (end 153.147444 98.5266) (width 0.3048) (layer F.Cu) (net 11))
-  (via (at 155.5496 102.3112) (size 0.762) (drill 0.4191) (layers F.Cu B.Cu) (net 11))
-  (segment (start 159.79138 106.55298) (end 155.5496 102.3112) (width 0.3048) (layer F.Cu) (net 11))
   (segment (start 159.79138 107.77222) (end 159.79138 106.55298) (width 0.3048) (layer F.Cu) (net 11))
   (segment (start 159.79138 107.77222) (end 159.79138 100.71098) (width 0.3048) (layer F.Cu) (net 11))
   (segment (start 159.79138 123.793964) (end 159.79138 107.77222) (width 0.3048) (layer F.Cu) (net 11))
-  (segment (start 153.2322 102.3112) (end 153.154 102.233) (width 0.3048) (layer B.Cu) (net 11) (status 30))
-  (segment (start 155.5496 102.3112) (end 153.2322 102.3112) (width 0.3048) (layer B.Cu) (net 11) (status 20))
   (segment (start 137.650725 100.304601) (end 142.870639 100.304601) (width 0.3048) (layer F.Cu) (net 11))
   (segment (start 125.2698 112.9792) (end 125.2698 112.0042) (width 0.3048) (layer F.Cu) (net 11) (status 10))
@@
   (segment (start 147.51361 95.96839) (end 146.054 97.428) (width 0.2032) (layer B.Cu) (net 15) (status 20))
   (segment (start 154.686 91.7448) (end 150.46241 95.96839) (width 0.2032) (layer B.Cu) (net 15) (status 10))
-  (segment (start 150.46241 95.96839) (end 147.51361 95.96839) (width 0.2032) (layer B.Cu) (net 15))
-  (segment (start 151.112108 99.13761) (end 152.586718 97.663) (width 0.2032) (layer B.Cu) (net 15))
-  (segment (start 146.46041 99.13761) (end 151.112108 99.13761) (width 0.2032) (layer B.Cu) (net 15))
-  (segment (start 146.054 97.553) (end 146.054 98.7312) (width 0.2032) (layer B.Cu) (net 15) (status 10))
-  (segment (start 146.054 98.7312) (end 146.46041 99.13761) (width 0.2032) (layer B.Cu) (net 15))
-  (segment (start 152.586718 97.663) (end 158.7754 97.663) (width 0.2032) (layer B.Cu) (net 15))
   (segment (start 158.7754 97.663) (end 160.5534 99.441) (width 0.2032) (layer B.Cu) (net 15))
   (via (at 159.5882 125.857) (size 0.762) (drill 0.4191) (layers F.Cu B.Cu) (net 15))
@@
   (segment (start 160.5534 104.6734) (end 160.5534 124.8918) (width 0.2032) (layer B.Cu) (net 15))
   (segment (start 160.5534 99.441) (end 160.5534 104.6734) (width 0.2032) (layer B.Cu) (net 15))
+  (segment (start 153.04219 95.96839) (end 150.00521 95.96839) (width 0.2032) (layer B.Cu) (net 15))
+  (segment (start 153.8224 96.7486) (end 153.04219 95.96839) (width 0.2032) (layer B.Cu) (net 15))
+  (segment (start 150.46241 95.96839) (end 150.00521 95.96839) (width 0.2032) (layer B.Cu) (net 15))
+  (segment (start 150.00521 95.96839) (end 147.51361 95.96839) (width 0.2032) (layer B.Cu) (net 15))
+  (segment (start 153.8478 96.7486) (end 154.7622 97.663) (width 0.2032) (layer B.Cu) (net 15))
+  (segment (start 154.7622 97.663) (end 158.7754 97.663) (width 0.2032) (layer B.Cu) (net 15))
   (segment (start 156.351401 96.562601) (end 154.6098 94.821) (width 0.2032) (layer F.Cu) (net 16) (status 20))
   (segment (start 152.14099 133.5278) (end 152.16639 133.5024) (width 0.2032) (layer F.Cu) (net 16))
@@
   (segment (start 151.6478 114.5172) (end 151.7478 114.5172) (width 0.2032) (layer B.Cu) (net 33) (status 30))
   (segment (start 151.7478 114.5172) (end 152.753401 113.511599) (width 0.2032) (layer B.Cu) (net 33) (status 10))
-  (segment (start 155.853399 113.511599) (end 157.0228 114.681) (width 0.2032) (layer B.Cu) (net 33))
   (segment (start 149.904 119.653) (end 149.804 119.653) (width 0.2032) (layer B.Cu) (net 33) (status 30))
   (segment (start 153.779683 118.888601) (end 153.538481 118.647399) (width 0.2032) (layer B.Cu) (net 33))
@@
   (segment (start 138.5316 113.7412) (end 139.4206 113.7412) (width 0.2032) (layer B.Cu) (net 33) (status 10))
   (segment (start 139.4206 113.7412) (end 142.9258 117.2464) (width 0.2032) (layer B.Cu) (net 33))
-  (segment (start 142.9258 117.2464) (end 149.1742 117.2464) (width 0.2032) (layer B.Cu) (net 33))
   (segment (start 151.514999 118.647399) (end 150.909601 118.647399) (width 0.2032) (layer B.Cu) (net 33))
   (segment (start 149.1742 117.2464) (end 150.575199 118.647399) (width 0.2032) (layer B.Cu) (net 33))
   (segment (start 128.1096 116.297648) (end 126.873476 115.061524) (width 0.2032) (layer F.Cu) (net 33))
   (segment (start 128.1096 117.3112) (end 128.1096 116.297648) (width 0.2032) (layer F.Cu) (net 33) (status 10))
+  (segment (start 156.4894 108.508318) (end 156.4894 114.1476) (width 0.2032) (layer B.Cu) (net 33))
+  (segment (start 154.438481 106.457399) (end 156.4894 108.508318) (width 0.2032) (layer B.Cu) (net 33))
+  (segment (start 155.853399 113.511599) (end 156.4894 114.1476) (width 0.2032) (layer B.Cu) (net 33))
+  (segment (start 156.4894 114.1476) (end 157.0228 114.681) (width 0.2032) (layer B.Cu) (net 33))
+  (segment (start 149.2016 102.233) (end 148.844 102.5906) (width 0.2032) (layer B.Cu) (net 33))
+  (segment (start 148.844 102.5906) (end 148.844 105.3084) (width 0.2032) (layer B.Cu) (net 33))
+  (segment (start 148.844 105.3084) (end 149.992999 106.457399) (width 0.2032) (layer B.Cu) (net 33))
+  (segment (start 149.992999 106.457399) (end 154.438481 106.457399) (width 0.2032) (layer B.Cu) (net 33))
+  (segment (start 153.154 102.233) (end 149.2016 102.233) (width 0.2032) (layer B.Cu) (net 33) (status 10))
+  (segment (start 148.49923 117.2464) (end 147.828 117.2464) (width 0.2032) (layer B.Cu) (net 33))
+  (segment (start 149.0726 116.67303) (end 148.49923 117.2464) (width 0.2032) (layer B.Cu) (net 33))
+  (segment (start 149.0726 115.5954) (end 149.0726 116.67303) (width 0.2032) (layer B.Cu) (net 33) (status 10))
+  (segment (start 142.9258 117.2464) (end 147.828 117.2464) (width 0.2032) (layer B.Cu) (net 33))
+  (segment (start 147.828 117.2464) (end 149.1742 117.2464) (width 0.2032) (layer B.Cu) (net 33))
   (segment (start 107.5794 106.5238) (end 108.4326 106.5238) (width 0.2032) (layer B.Cu) (net 34) (status 20))
   (segment (start 106.700799 105.645199) (end 107.5794 106.5238) (width 0.2032) (layer B.Cu) (net 34))
