File: design/spidey_sense_v2.0/Amplifier.kicad_sch (KiCad schematic)
At the start: 5 parts, among them U6 LT1001

Commit message: Updated footprints
Parts:
- U3: renamed from U6; footprint SamacSys_Parts:NE555DR -> Package_SO:SOP-8_3.9x4.9mm_P1.27mm
- renumbered C10 to C1, C11 to C2, R8 to R4, R9 to R5
Changed lines of the file:
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@@
   (symbol (lib_id "Device:R") (at 127 93.98 180)
     (in_bom yes) (on_board yes)
-    (property "Reference" "R8" (id 0) (at 130.81 92.71 0))
+    (property "Reference" "R4" (id 0) (at 130.81 92.71 0))
     (property "Value" "1kΩ" (id 1) (at 130.81 95.25 0))
     (property "Footprint" "Resistor_SMD:R_0805_2012Metric_Pad1.20x1.40mm_HandSolder" (id 2) (at 128.778 93.98 90)
@@
   (symbol (lib_id "Device:C") (at 133.35 115.57 0)
     (in_bom yes) (on_board yes)
-    (property "Reference" "C10" (id 0) (at 136.271 114.4016 0)
+    (property "Reference" "C1" (id 0) (at 136.271 114.4016 0)
       (effects (font (size 1.27 1.27)) (justify left))
     )
@@
   (symbol (lib_id "Device:C") (at 152.4 88.9 270)
     (in_bom yes) (on_board yes)
-    (property "Reference" "C11" (id 0) (at 153.5684 91.821 90)
+    (property "Reference" "C2" (id 0) (at 153.5684 91.821 90)
       (effects (font (size 1.27 1.27)) (justify left))
     )
@@
   (symbol (lib_id "power:GND") (at 133.35 120.65 0)
     (in_bom yes) (on_board yes)
-    (property "Reference" "#PWR026" (id 0) (at 133.35 127 0)
+    (property "Reference" "#PWR09" (id 0) (at 133.35 127 0)
       (effects (font (size 1.27 1.27)) hide)
     )
@@
   (symbol (lib_id "power:GND") (at 127 99.06 0)
     (in_bom yes) (on_board yes)
-    (property "Reference" "#PWR025" (id 0) (at 127 105.41 0)
+    (property "Reference" "#PWR03" (id 0) (at 127 105.41 0)
       (effects (font (size 1.27 1.27)) hide)
     )
@@
   (symbol (lib_id "Device:R") (at 152.4 83.82 270)
     (in_bom yes) (on_board yes)
-    (property "Reference" "R9" (id 0) (at 152.4 78.5622 90))
+    (property "Reference" "R5" (id 0) (at 152.4 78.5622 90))
     (property "Value" "17.3kΩ" (id 1) (at 152.4 80.8736 90))
     (property "Footprint" "Resistor_SMD:R_0805_2012Metric_Pad1.20x1.40mm_HandSolder" (id 2) (at 152.4 82.042 90)
@@
   (symbol (lib_id "power:+5V") (at 144.78 96.52 0)
     (in_bom yes) (on_board yes)
-    (property "Reference" "#PWR027" (id 0) (at 144.78 100.33 0)
+    (property "Reference" "#PWR010" (id 0) (at 144.78 100.33 0)
       (effects (font (size 1.27 1.27)) hide)
     )
@@
   (symbol (lib_id "power:-5V") (at 151.13 115.57 0)
     (in_bom yes) (on_board yes)
-    (property "Reference" "#PWR028" (id 0) (at 151.13 113.03 0)
+    (property "Reference" "#PWR011" (id 0) (at 151.13 113.03 0)
       (effects (font (size 1.27 1.27)) hide)
     )
@@
   (symbol (lib_id "Thermocouple:LT1001") (at 142.24 105.41 270)
     (in_bom yes) (on_board yes)
-    (property "Reference" "U6" (id 0) (at 156.0576 104.2416 90)
+    (property "Reference" "U3" (id 0) (at 156.0576 104.2416 90)
       (effects (font (size 1.27 1.27)) (justify left))
     )
@@
       (effects (font (size 1.27 1.27)) (justify left))
     )
-    (property "Footprint" "SamacSys_Parts:NE555DR" (id 2) (at 142.24 105.41 0)
+    (property "Footprint" "Package_SO:SOP-8_3.9x4.9mm_P1.27mm" (id 2) (at 142.24 105.41 0)
       (effects (font (size 1.27 1.27)) hide)
     )

Commit message: Updated PCB
Parts:
- renumbered C1 to C10, C2 to C11, R4 to R8, R5 to R9, U3 to U6
Changed lines of the file:
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@@
   (symbol (lib_id "Device:R") (at 127 93.98 180)
     (in_bom yes) (on_board yes)
-    (property "Reference" "R4" (id 0) (at 130.81 92.71 0))
+    (property "Reference" "R8" (id 0) (at 130.81 92.71 0))
     (property "Value" "1kΩ" (id 1) (at 130.81 95.25 0))
     (property "Footprint" "Resistor_SMD:R_0805_2012Metric_Pad1.20x1.40mm_HandSolder" (id 2) (at 128.778 93.98 90)
@@
   (symbol (lib_id "Device:C") (at 133.35 115.57 0)
     (in_bom yes) (on_board yes)
-    (property "Reference" "C1" (id 0) (at 136.271 114.4016 0)
+    (property "Reference" "C10" (id 0) (at 136.271 114.4016 0)
       (effects (font (size 1.27 1.27)) (justify left))
     )
@@
   (symbol (lib_id "Device:C") (at 152.4 88.9 270)
     (in_bom yes) (on_board yes)
-    (property "Reference" "C2" (id 0) (at 153.5684 91.821 90)
+    (property "Reference" "C11" (id 0) (at 153.5684 91.821 90)
       (effects (font (size 1.27 1.27)) (justify left))
     )
@@
   (symbol (lib_id "power:GND") (at 133.35 120.65 0)
     (in_bom yes) (on_board yes)
-    (property "Reference" "#PWR09" (id 0) (at 133.35 127 0)
+    (property "Reference" "#PWR026" (id 0) (at 133.35 127 0)
       (effects (font (size 1.27 1.27)) hide)
     )
@@
   (symbol (lib_id "power:GND") (at 127 99.06 0)
     (in_bom yes) (on_board yes)
-    (property "Reference" "#PWR03" (id 0) (at 127 105.41 0)
+    (property "Reference" "#PWR025" (id 0) (at 127 105.41 0)
       (effects (font (size 1.27 1.27)) hide)
     )
@@
   (symbol (lib_id "Device:R") (at 152.4 83.82 270)
     (in_bom yes) (on_board yes)
-    (property "Reference" "R5" (id 0) (at 152.4 78.5622 90))
+    (property "Reference" "R9" (id 0) (at 152.4 78.5622 90))
     (property "Value" "17.3kΩ" (id 1) (at 152.4 80.8736 90))
     (property "Footprint" "Resistor_SMD:R_0805_2012Metric_Pad1.20x1.40mm_HandSolder" (id 2) (at 152.4 82.042 90)
@@
   (symbol (lib_id "power:+5V") (at 144.78 96.52 0)
     (in_bom yes) (on_board yes)
-    (property "Reference" "#PWR010" (id 0) (at 144.78 100.33 0)
+    (property "Reference" "#PWR027" (id 0) (at 144.78 100.33 0)
       (effects (font (size 1.27 1.27)) hide)
     )
@@
   (symbol (lib_id "power:-5V") (at 151.13 115.57 0)
     (in_bom yes) (on_board yes)
-    (property "Reference" "#PWR011" (id 0) (at 151.13 113.03 0)
+    (property "Reference" "#PWR028" (id 0) (at 151.13 113.03 0)
       (effects (font (size 1.27 1.27)) hide)
     )
@@
   (symbol (lib_id "Thermocouple:LT1001") (at 142.24 105.41 270)
     (in_bom yes) (on_board yes)
-    (property "Reference" "U3" (id 0) (at 156.0576 104.2416 90)
+    (property "Reference" "U6" (id 0) (at 156.0576 104.2416 90)
       (effects (font (size 1.27 1.27)) (justify left))
     )
