File: design/power_board/power_board.kicad_sch (KiCad schematic)
At the start: 8 parts, among them J1 Screw_Terminal_01x02, J2 Screw_Terminal_01x02, J3 Screw_Terminal_01x03

Commit message: Update power_board.kicad_sch
Other:
- note added: "24V from GSPD"
- note removed: "6S lipo (19.2 - 25.2V) or 24V AC/DC adapter"
Changed lines of the file:
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@@
     (effects (font (size 1.27 1.27)) (justify right bottom))
   )
-  (text "6S lipo (19.2 - 25.2V)\nor 24V AC/DC adapter" (at 68.58 35.56 0)
+  (text "24V from GSPD" (at 68.58 35.56 0)
     (effects (font (size 1.27 1.27)) (justify right bottom))
   )

Commit message: i
Other:
- moved on the sheet: J1, J2, J3, R1, R2, R3, R4
