File: design/power_board/buck.kicad_sch (KiCad schematic)
At the start: 9 parts, among them U1 LV2862YDDCR

Commit message: changed resistor value
Parts:
- R2: value 277.58k -> _k
Changed lines of the file:
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@@
       (effects (font (size 1.27 1.27)) (justify left))
     )
-    (property "Value" "277.58k" (at 176.9872 100.203 0)
+    (property "Value" "_k" (at 176.9872 100.203 0)
       (effects (font (size 1.27 1.27)) (justify left))
     )
