File: design/thermocouple_board/thermocouple.kicad_sch (KiCad schematic)
At the start: 6 parts, among them J5 Thermocouple conn, U3 MAX31855KASA

Commit message: Added optional can termination resistor
Parts:
- renumbered C6 to C10, C5 to C9, L2 to L3, L1 to L4, U3 to U5
Changed lines of the file:
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@@
   (symbol (lib_id "Device:L_Ferrite_Small") (at 107.95 110.49 90) (unit 1)
     (in_bom yes) (on_board yes) (dnp no)
-    (property "Reference" "L1" (at 107.95 111.76 90)
+    (property "Reference" "L4" (at 107.95 111.76 90)
       (effects (font (size 1.27 1.27)))
     )
@@
       (project "thermocouple_board"
         (path "/bddc1c86-7e70-444c-8c58-d2a4afd414ff/196db3b3-bb6e-4aaa-bfdb-62271ec88ddc"
-          (reference "L1") (unit 1)
-        )
-        (path "/bddc1c86-7e70-444c-8c58-d2a4afd414ff/63a9e4b5-6489-403b-b271-ab052f2c16d6"
           (reference "L4") (unit 1)
+        )
+        (path "/bddc1c86-7e70-444c-8c58-d2a4afd414ff/63a9e4b5-6489-403b-b271-ab052f2c16d6"
+          (reference "L2") (unit 1)
         )
         (path "/bddc1c86-7e70-444c-8c58-d2a4afd414ff/83e96294-8b9a-4632-a548-e13053a6ac34"
@@
   (symbol (lib_id "power:GND") (at 172.72 90.17 0) (unit 1)
     (in_bom yes) (on_board yes) (dnp no) (fields_autoplaced)
-    (property "Reference" "#PWR023" (at 172.72 96.52 0)
+    (property "Reference" "#PWR030" (at 172.72 96.52 0)
       (effects (font (size 1.27 1.27)) hide)
     )
@@
       (project "thermocouple_board"
         (path "/bddc1c86-7e70-444c-8c58-d2a4afd414ff/196db3b3-bb6e-4aaa-bfdb-62271ec88ddc"
-          (reference "#PWR023") (unit 1)
-        )
-        (path "/bddc1c86-7e70-444c-8c58-d2a4afd414ff/63a9e4b5-6489-403b-b271-ab052f2c16d6"
           (reference "#PWR030") (unit 1)
+        )
+        (path "/bddc1c86-7e70-444c-8c58-d2a4afd414ff/63a9e4b5-6489-403b-b271-ab052f2c16d6"
+          (reference "#PWR026") (unit 1)
         )
         (path "/bddc1c86-7e70-444c-8c58-d2a4afd414ff/83e96294-8b9a-4632-a548-e13053a6ac34"
@@
   (symbol (lib_id "Device:C_Small") (at 115.57 107.95 0) (unit 1)
     (in_bom yes) (on_board yes) (dnp no)
-    (property "Reference" "C5" (at 118.11 106.68 0)
+    (property "Reference" "C9" (at 118.11 106.68 0)
       (effects (font (size 1.27 1.27)) (justify left))
     )
@@
       (project "thermocouple_board"
         (path "/bddc1c86-7e70-444c-8c58-d2a4afd414ff/196db3b3-bb6e-4aaa-bfdb-62271ec88ddc"
-          (reference "C5") (unit 1)
-        )
-        (path "/bddc1c86-7e70-444c-8c58-d2a4afd414ff/63a9e4b5-6489-403b-b271-ab052f2c16d6"
           (reference "C9") (unit 1)
         )
+        (path "/bddc1c86-7e70-444c-8c58-d2a4afd414ff/63a9e4b5-6489-403b-b271-ab052f2c16d6"
+          (reference "C7") (unit 1)
+        )
         (path "/bddc1c86-7e70-444c-8c58-d2a4afd414ff/83e96294-8b9a-4632-a548-e13053a6ac34"
           (reference "C11") (unit 1)
@@
   (symbol (lib_id "power:+3.3V") (at 172.72 85.09 0) (unit 1)
     (in_bom yes) (on_board yes) (dnp no) (fields_autoplaced)
-    (property "Reference" "#PWR022" (at 172.72 88.9 0)
+    (property "Reference" "#PWR029" (at 172.72 88.9 0)
       (effects (font (size 1.27 1.27)) hide)
     )
@@
       (project "thermocouple_board"
         (path "/bddc1c86-7e70-444c-8c58-d2a4afd414ff/196db3b3-bb6e-4aaa-bfdb-62271ec88ddc"
-          (reference "#PWR022") (unit 1)
-        )
-        (path "/bddc1c86-7e70-444c-8c58-d2a4afd414ff/63a9e4b5-6489-403b-b271-ab052f2c16d6"
           (reference "#PWR029") (unit 1)
         )
+        (path "/bddc1c86-7e70-444c-8c58-d2a4afd414ff/63a9e4b5-6489-403b-b271-ab052f2c16d6"
+          (reference "#PWR025") (unit 1)
+        )
         (path "/bddc1c86-7e70-444c-8c58-d2a4afd414ff/83e96294-8b9a-4632-a548-e13053a6ac34"
           (reference "#PWR033") (unit 1)
@@
   (symbol (lib_id "Sensor_Temperature:MAX31855KASA") (at 152.4 101.6 0) (unit 1)
     (in_bom yes) (on_board yes) (dnp no) (fields_autoplaced)
-    (property "Reference" "U3" (at 143.51 88.9 0)
+    (property "Reference" "U5" (at 143.51 88.9 0)
       (effects (font (size 1.27 1.27)) (justify left))
     )
@@
       (project "thermocouple_board"
         (path "/bddc1c86-7e70-444c-8c58-d2a4afd414ff/196db3b3-bb6e-4aaa-bfdb-62271ec88ddc"
-          (reference "U3") (unit 1)
-        )
-        (path "/bddc1c86-7e70-444c-8c58-d2a4afd414ff/63a9e4b5-6489-403b-b271-ab052f2c16d6"
           (reference "U5") (unit 1)
+        )
+        (path "/bddc1c86-7e70-444c-8c58-d2a4afd414ff/63a9e4b5-6489-403b-b271-ab052f2c16d6"
+          (reference "U4") (unit 1)
         )
         (path "/bddc1c86-7e70-444c-8c58-d2a4afd414ff/83e96294-8b9a-4632-a548-e13053a6ac34"
@@
   (symbol (lib_id "Device:L_Ferrite_Small") (at 107.95 105.41 90) (unit 1)
     (in_bom yes) (on_board yes) (dnp no)
-    (property "Reference" "L2" (at 107.95 99.06 90)
+    (property "Reference" "L3" (at 107.95 99.06 90)
       (effects (font (size 1.27 1.27)))
     )
@@
       (project "thermocouple_board"
         (path "/bddc1c86-7e70-444c-8c58-d2a4afd414ff/196db3b3-bb6e-4aaa-bfdb-62271ec88ddc"
-          (reference "L2") (unit 1)
-        )
-        (path "/bddc1c86-7e70-444c-8c58-d2a4afd414ff/63a9e4b5-6489-403b-b271-ab052f2c16d6"
           (reference "L3") (unit 1)
+        )
+        (path "/bddc1c86-7e70-444c-8c58-d2a4afd414ff/63a9e4b5-6489-403b-b271-ab052f2c16d6"
+          (reference "L1") (unit 1)
         )
         (path "/bddc1c86-7e70-444c-8c58-d2a4afd414ff/83e96294-8b9a-4632-a548-e13053a6ac34"
@@
   (symbol (lib_id "power:+3.3V") (at 165.1 92.71 0) (unit 1)
     (in_bom yes) (on_board yes) (dnp no) (fields_autoplaced)
-    (property "Reference" "#PWR020" (at 165.1 96.52 0)
+    (property "Reference" "#PWR027" (at 165.1 96.52 0)
       (effects (font (size 1.27 1.27)) hide)
     )
@@
       (project "thermocouple_board"
         (path "/bddc1c86-7e70-444c-8c58-d2a4afd414ff/196db3b3-bb6e-4aaa-bfdb-62271ec88ddc"
-          (reference "#PWR020") (unit 1)
-        )
-        (path "/bddc1c86-7e70-444c-8c58-d2a4afd414ff/63a9e4b5-6489-403b-b271-ab052f2c16d6"
           (reference "#PWR027") (unit 1)
         )
+        (path "/bddc1c86-7e70-444c-8c58-d2a4afd414ff/63a9e4b5-6489-403b-b271-ab052f2c16d6"
+          (reference "#PWR023") (unit 1)
+        )
         (path "/bddc1c86-7e70-444c-8c58-d2a4afd414ff/83e96294-8b9a-4632-a548-e13053a6ac34"
           (reference "#PWR031") (unit 1)
@@
   (symbol (lib_id "power:GND") (at 165.1 113.03 0) (unit 1)
     (in_bom yes) (on_board yes) (dnp no) (fields_autoplaced)
-    (property "Reference" "#PWR021" (at 165.1 119.38 0)
+    (property "Reference" "#PWR028" (at 165.1 119.38 0)
       (effects (font (size 1.27 1.27)) hide)
     )
@@
       (project "thermocouple_board"
         (path "/bddc1c86-7e70-444c-8c58-d2a4afd414ff/196db3b3-bb6e-4aaa-bfdb-62271ec88ddc"
-          (reference "#PWR021") (unit 1)
-        )
-        (path "/bddc1c86-7e70-444c-8c58-d2a4afd414ff/63a9e4b5-6489-403b-b271-ab052f2c16d6"
           (reference "#PWR028") (unit 1)
+        )
+        (path "/bddc1c86-7e70-444c-8c58-d2a4afd414ff/63a9e4b5-6489-403b-b271-ab052f2c16d6"
+          (reference "#PWR024") (unit 1)
         )
         (path "/bddc1c86-7e70-444c-8c58-d2a4afd414ff/83e96294-8b9a-4632-a548-e13053a6ac34"
@@
   (symbol (lib_id "Device:C_Small") (at 172.72 87.63 0) (unit 1)
     (in_bom yes) (on_board yes) (dnp no)
-    (property "Reference" "C6" (at 175.26 86.36 0)
+    (property "Reference" "C10" (at 175.26 86.36 0)
       (effects (font (size 1.27 1.27)) (justify left))
     )
@@
       (project "thermocouple_board"
         (path "/bddc1c86-7e70-444c-8c58-d2a4afd414ff/196db3b3-bb6e-4aaa-bfdb-62271ec88ddc"
-          (reference "C6") (unit 1)
-        )
-        (path "/bddc1c86-7e70-444c-8c58-d2a4afd414ff/63a9e4b5-6489-403b-b271-ab052f2c16d6"
           (reference "C10") (unit 1)
         )
-        (path "/bddc1c86-7e70-444c-8c58-d2a4afd414ff/83e96294-8b9a-4632-a548-e13053a6ac34"
+        (path "/bddc1c86-7e70-444c-8c58-d2a4afd414ff/63a9e4b5-6489-403b-b271-ab052f2c16d6"
+          (reference "C8") (unit 1)
+        )
+        (path "/bddc1c86-7e70-444c-8c58-d2a4afd414ff/83e96294-8b9a-4632-a548-e13053a6ac34"

Commit message: Addressed Artem's comments
Parts:
- C10: value 0.01uF -> 0.1uF; footprint (none) -> Capacitor_SMD:C_0805_2012Metric_Pad1.18x1.45mm_HandSolder
- C9: footprint (none) -> Capacitor_SMD:C_0805_2012Metric_Pad1.18x1.45mm_HandSolder
Connections:
- net SCK renamed SCLK_3V3
- net SDO renamed MISO_3V3
Other:
- moved on the sheet: L3, L4

Commit message: Addressed comments added 3.3V PIC
Parts:
- C9: value 0.01uF -> 0.1uF
Connections:
- net MISO_3V3 renamed MISO
- net SCLK_3V3 renamed SCLK

Commit message: Added footprints
Parts:
- J5: footprint (none) -> TerminalBlock_Phoenix:TerminalBlock_Phoenix_MKDS-1,5-2-5.08_1x02_P5.08mm_Horizontal
Changed lines of the file:
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@@
       (effects (font (size 1.27 1.27)))
     )
-    (property "Footprint" "" (at 85.09 110.49 0)
+    (property "Footprint" "TerminalBlock_Phoenix:TerminalBlock_Phoenix_MKDS-1,5-2-5.08_1x02_P5.08mm_Horizontal" (at 85.09 110.49 0)
       (effects (font (size 1.27 1.27)) hide)
     )

Commit message: Addressed comments
Connections:
- net at L4.1: now also J5.2 (Pin_2); no longer J5.1 (Pin_1)
- net at L3.1: now also J5.1 (Pin_1); no longer J5.2 (Pin_2)
Other:
- moved on the sheet: J5
Changed lines of the file:
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@@
     )
   )
-  (symbol (lib_id "Connector:Screw_Terminal_01x02") (at 85.09 110.49 180) (unit 1)
+  (symbol (lib_id "Connector:Screw_Terminal_01x02") (at 85.09 107.95 0) (mirror y) (unit 1)
     (in_bom yes) (on_board yes) (dnp no)
     (property "Reference" "J5" (at 85.09 101.6 0)
@@
       (effects (font (size 1.27 1.27)))
     )
-    (property "Footprint" "TerminalBlock_Phoenix:TerminalBlock_Phoenix_MKDS-1,5-2-5.08_1x02_P5.08mm_Horizontal" (at 85.09 110.49 0)
+    (property "Footprint" "TerminalBlock_Phoenix:TerminalBlock_Phoenix_MKDS-1,5-2-5.08_1x02_P5.08mm_Horizontal" (at 85.09 107.95 0)
       (effects (font (size 1.27 1.27)) hide)
     )
-    (property "Datasheet" "~" (at 85.09 110.49 0)
+    (property "Datasheet" "~" (at 85.09 107.95 0)
       (effects (font (size 1.27 1.27)) hide)
     )
