File: design/thermocouple_board/thermocouple_board.kicad_sch (KiCad schematic)
At the start: 24 parts, among them J1 Prog Conn, J2 CAN Conn, J3 CAN Ext Conn, U1 PIC18F26K83, U2 MCP2562, U4 AP2120N-3.3TRG1, Y1 12 MHz

Commit message: Renamed SDI tag to SDO
Connections:
- net SDI renamed SDO
Other:
- note added: "Add optional can termination resistor?"
- note added: "This PIC uses 3 wire SPI. RC4 can either send or receive data"
- note removed: "Add optional can termination resistor"
Changed lines of the file:
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@@
     (stroke (width 0) (type default))
   )
-  (text "Add optional can termination resistor\n" (at 132.08 139.7 0)
+  (text "Add optional can termination resistor?\n" (at 132.08 139.7 0)
+    (effects (font (size 1.27 1.27)) (justify left bottom))
+  )
+  (text "This PIC uses 3 wire SPI. RC4 \ncan either send or receive data"
+    (at 48.26 116.84 0)
     (effects (font (size 1.27 1.27)) (justify left bottom))
   )
@@
     (effects (font (size 1.27 1.27)) (justify left bottom))
   )
-  (label "SDI" (at 213.36 86.36 180) (fields_autoplaced)
+  (label "SDO" (at 213.36 86.36 180) (fields_autoplaced)
     (effects (font (size 1.27 1.27)) (justify right bottom))
   )
-  (label "SDI" (at 213.36 109.22 180) (fields_autoplaced)
+  (label "SDO" (at 213.36 109.22 180) (fields_autoplaced)
     (effects (font (size 1.27 1.27)) (justify right bottom))
   )
@@
     (effects (font (size 1.27 1.27)) (justify right bottom))
   )
-  (label "SDI" (at 213.36 63.5 180) (fields_autoplaced)
+  (label "SDO" (at 213.36 63.5 180) (fields_autoplaced)
     (effects (font (size 1.27 1.27)) (justify right bottom))
   )
@@
     (effects (font (size 1.27 1.27)) (justify left bottom))
   )
-  (label "SDI" (at 213.36 132.08 180) (fields_autoplaced)
+  (label "SDO" (at 213.36 132.08 180) (fields_autoplaced)
     (effects (font (size 1.27 1.27)) (justify right bottom))
   )
-  (label "SDI" (at 86.36 114.3 180) (fields_autoplaced)
+  (label "SDO" (at 86.36 114.3 180) (fields_autoplaced)
     (effects (font (size 1.27 1.27)) (justify right bottom))
   )

Commit message: Added optional can termination resistor
Parts:
- added JP1: Jumper, symbol Jumper:Jumper_2_Open
- added R1: 120R, Resistor_SMD:R_0805_2012Metric_Pad1.20x1.40mm_HandSolder, symbol Device:R_US
- renumbered C7 to C5, C8 to C6, U4 to U3
Connections:
- net CANH: now also R1.2
- net CANL: now also JP1.2 (B)
- new net: JP1.1 (A), R1.1
Other:
- note removed: "Add optional can termination resistor?"

Commit message: Addressed Artem's comments
Parts:
- added D2 (x2): GREEN, LED_SMD:LED_1206_3216Metric_Pad1.42x1.75mm_HandSolder, symbol Device:LED
- added D6: 1.5KExxA, symbol Diode:1.5KExxA
- added R1: 220R, Resistor_SMD:R_0805_2012Metric_Pad1.20x1.40mm_HandSolder, symbol Device:R_US
- added R1: 120R, Resistor_SMD:R_0805_2012Metric_Pad1.20x1.40mm_HandSolder, symbol Device:R_US
- added R4 (x2): 10k, Resistor_SMD:R_0805_2012Metric_Pad1.20x1.40mm_HandSolder, symbol Device:R_US
- added TP1, TP2, TP3, TP4, TP5: TestPoint, TestPoint:TestPoint_Pad_2.0x2.0mm, symbol Connector:TestPoint
- added U8, U9: 74LVC1T45GW_125, turbopumpfydp_lib_footprints:SOP65P210X110-6N, symbol turbopumpfydp_lib:74LVC1T45GW_125
- C4: footprint (none) -> Capacitor_SMD:C_0805_2012Metric_Pad1.18x1.45mm_HandSolder
- C5: value 1uF -> 4.7uF; footprint (none) -> Capacitor_SMD:C_0805_2012Metric_Pad1.18x1.45mm_HandSolder
- C6: value 1uF -> 22uF; footprint (none) -> Capacitor_SMD:C_0805_2012Metric_Pad1.18x1.45mm_HandSolder
- JP1: footprint (none) -> Connector_PinHeader_2.54mm:PinHeader_1x02_P2.54mm_Vertical
- U1: footprint (none) -> Package_SO:SOIC-28W_7.5x17.9mm_P1.27mm
- U2: footprint (none) -> Package_SO:SOIC-8_3.9x4.9mm_P1.27mm
- U3: footprint (none) -> Package_TO_SOT_SMD:SOT-23-3
Connections:
- net +3.3V: now also D2.2 (A), TP2.1, U8.1 (VCC(A)), U9.6 (VCC(B))
- net +5V: now also D2.2 (A), D6.1 (A1), R4.1, R4.1, TP1.1, U8.6 (VCC(B)), U9.1 (VCC(A))
- net CAN_RX: now also TP5.1
- net CAN_TX: now also TP4.1
- net GND: now also D6.2 (A2), R1.2, R1.2, TP3.1, U8.2 (GND), U8.5 (DIR), U9.2 (GND), U9.5 (DIR)
- net SCK renamed SCLK
- net SCLK: now also R4.2, U8.4 (B)
- net SDO renamed MISO
- net MISO: now also R4.2, U9.3 (A)
- new net: D2.1 (K), R1.1 (x2)
- new net MISO_3V3: U9.4 (B)
- new net SCLK_3V3: U8.3 (A)
Other:
- sheet Thermocouple_1 ports: added none; removed SCK, SDO
- sheet Thermocouple_2 ports: added none; removed SCK, SDO
- sheet Thermocouple_3 ports: added none; removed SCK, SDO
- sheet Thermocouple_4 ports: added none; removed SCK, SDO
- note removed: "This PIC uses 3 wire SPI. RC4 can either send or receive data"
- moved on the sheet: C1, C2, C4, C5, C6, H1, H2, H3, H4, J1, J2, J3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

Commit message: Addressed comments added 3.3V PIC
Parts:
- removed D1: WHITE, LED_SMD:LED_1206_3216Metric_Pad1.42x1.75mm_HandSolder, symbol Device:LED
- removed U8, U9: 74LVC1T45GW_125, turbopumpfydp_lib_footprints:SOP65P210X110-6N, symbol turbopumpfydp_lib:74LVC1T45GW_125
- added D3: YELLOW, symbol Device:LED
- added R4 (x4): 10k, Resistor_SMD:R_0805_2012Metric_Pad1.20x1.40mm_HandSolder, symbol Device:R_US
- added TP6, TP7: TestPoint, symbol Connector:TestPoint
- D2: value BLUE -> ORANGE
- R3: value 220R -> 120R
- U1: value PIC18F26K83 -> PIC18LF26K83
- renumbered D6 to D1, TP5 to TP1, TP4 to TP2, TP1 to TP3, TP2 to TP4, TP3 to TP5
Connections:
- net +3.3V: now also C4.1, D2.2 (A), D3.2 (A), J1.2 (Pin_2), R4.1, R4.1, R4.1, U1.20 (VDD), U2.5 (VIO), D3.2 (A), R4.1, R4.1, R4.1, R4.1
- net +5V: no longer C4.1, D2.2 (A), D3.2 (A), J1.2 (Pin_2), R4.1, R4.1, R4.1, U1.20 (VDD), U2.5 (VIO)
- net CS1: now also R4.2
- net CS2: now also R4.2
- net CS3: now also R4.2
- net CS4: now also R4.2
- net MISO: now also TP6.1
- net SCLK: now also TP7.1
- net at R1.1: now also D3.1 (K)
Other:
- note added: "Connectors"
- note added: "MCU"
- note added: "Power"
- note added: "Thermocouples"
- moved on the sheet: C1, C2, C4, C5, C6, D2, D3, H1, H2, H3, H4, JP1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

Commit message: Added footprints
Parts:
- D1: footprint (none) -> Diode_SMD:D_SOD-523
- D3: footprint (none) -> LED_SMD:LED_1206_3216Metric_Pad1.42x1.75mm_HandSolder
- J1: footprint (none) -> canhw:PinHeader_5x2.54_SMD_90deg_952-3198-1-ND
- J2, J3: footprint (none) -> TerminalBlock_Phoenix:TerminalBlock_Phoenix_MKDS-1,5-4-5.08_1x04_P5.08mm_Horizontal
- TP6, TP7: footprint (none) -> TestPoint:TestPoint_Pad_2.0x2.0mm
Changed lines of the file:
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@@
       (effects (font (size 1.27 1.27)) (justify left))
     )
-    (property "Footprint" "" (at 115.57 40.64 0)
+    (property "Footprint" "TerminalBlock_Phoenix:TerminalBlock_Phoenix_MKDS-1,5-4-5.08_1x04_P5.08mm_Horizontal" (at 115.57 40.64 0)
       (effects (font (size 1.27 1.27)) hide)
     )
@@
       (effects (font (size 1.27 1.27)) (justify left))
     )
-    (property "Footprint" "" (at 69.85 40.64 0)
+    (property "Footprint" "TerminalBlock_Phoenix:TerminalBlock_Phoenix_MKDS-1,5-4-5.08_1x04_P5.08mm_Horizontal" (at 69.85 40.64 0)
       (effects (font (size 1.27 1.27)) hide)
     )
@@
       (effects (font (size 1.27 1.27)) (justify right))
     )
-    (property "Footprint" "" (at 60.96 120.65 0)
+    (property "Footprint" "TestPoint:TestPoint_Pad_2.0x2.0mm" (at 60.96 120.65 0)
       (effects (font (size 1.27 1.27)) hide)
     )
@@
       (effects (font (size 1.27 1.27)) (justify right))
     )
-    (property "Footprint" "" (at 152.4 78.74 0)
+    (property "Footprint" "LED_SMD:LED_1206_3216Metric_Pad1.42x1.75mm_HandSolder" (at 152.4 78.74 0)
       (effects (font (size 1.27 1.27)) hide)
     )
@@
       (effects (font (size 1.27 1.27)) (justify left))
     )
-    (property "Footprint" "" (at 39.37 43.18 0)
+    (property "Footprint" "canhw:PinHeader_5x2.54_SMD_90deg_952-3198-1-ND" (at 39.37 43.18 0)
       (effects (font (size 1.27 1.27)) hide)
     )
@@
       (effects (font (size 1.27 1.27)) (justify left))
     )
-    (property "Footprint" "" (at 82.55 41.91 0)
+    (property "Footprint" "Diode_SMD:D_SOD-523" (at 82.55 41.91 0)
       (effects (font (size 1.27 1.27)) hide)
     )
@@
       (effects (font (size 1.27 1.27)) (justify right))
     )
-    (property "Footprint" "" (at 74.93 120.65 0)
-      (effects (font (size 1.27 1.27)) hide)
-    )
+    (property "Footprint" "TestPoint:TestPoint_Pad_2.0x2.0mm" (at 74.93 120.65 0)
+      (effects (font (size 1.27 1.27)) hide)
+    )

Commit message: Finished routing, still need to add logo
Connections:
- net +5V: now also J3.4 (Pin_4); no longer J3.1 (Pin_1)
- net CANH: now also J3.3 (Pin_3); no longer J3.2 (Pin_2)
- net CANL: now also J3.2 (Pin_2); no longer J3.3 (Pin_3)
- net GND: now also J3.1 (Pin_1); no longer J3.4 (Pin_4)
Other:
- moved on the sheet: J3
Changed lines of the file:
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@@
     )
   )
-  (symbol (lib_id "Connector:Screw_Terminal_01x04") (at 115.57 40.64 0) (mirror y) (unit 1)
+  (symbol (lib_id "Connector:Screw_Terminal_01x04") (at 115.57 43.18 180) (unit 1)
     (in_bom yes) (on_board yes) (dnp no)
     (property "Reference" "J3" (at 116.84 31.75 0)
@@
       (effects (font (size 1.27 1.27)) (justify left))
     )
-    (property "Footprint" "TerminalBlock_Phoenix:TerminalBlock_Phoenix_MKDS-1,5-4-5.08_1x04_P5.08mm_Horizontal" (at 115.57 40.64 0)
+    (property "Footprint" "TerminalBlock_Phoenix:TerminalBlock_Phoenix_MKDS-1,5-4-5.08_1x04_P5.08mm_Horizontal" (at 115.57 43.18 0)
       (effects (font (size 1.27 1.27)) hide)
     )
-    (property "Datasheet" "~" (at 115.57 40.64 0)
+    (property "Datasheet" "~" (at 115.57 43.18 0)
       (effects (font (size 1.27 1.27)) hide)
     )

Commit message: Addressed comments
Parts:
- TP1, TP2, TP3, TP4, TP5, TP6, TP7: footprint TestPoint:TestPoint_Pad_2.0x2.0mm -> TestPoint:TestPoint_Keystone_5005-5009_Compact
Connections:
- net +5V: now also J2.4 (Pin_4), J3.1 (Pin_1); no longer J2.1 (Pin_1), J3.4 (Pin_4)
- net CANH: now also J2.3 (Pin_3), J3.2 (Pin_2); no longer J2.2 (Pin_2), J3.3 (Pin_3)
- net CANL: now also J2.2 (Pin_2), J3.3 (Pin_3); no longer J2.3 (Pin_3), J3.2 (Pin_2)
- net GND: now also J2.1 (Pin_1), J3.4 (Pin_4); no longer J2.4 (Pin_4), J3.1 (Pin_1)
Other:
- moved on the sheet: J2, J3
Changed lines of the file:
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@@
     )
   )
-  (symbol (lib_id "Connector:Screw_Terminal_01x04") (at 115.57 43.18 180) (unit 1)
+  (symbol (lib_id "Connector:Screw_Terminal_01x04") (at 115.57 40.64 0) (mirror y) (unit 1)
     (in_bom yes) (on_board yes) (dnp no)
     (property "Reference" "J3" (at 116.84 31.75 0)
@@
       (effects (font (size 1.27 1.27)) (justify left))
     )
-    (property "Footprint" "TerminalBlock_Phoenix:TerminalBlock_Phoenix_MKDS-1,5-4-5.08_1x04_P5.08mm_Horizontal" (at 115.57 43.18 0)
-      (effects (font (size 1.27 1.27)) hide)
-    )
-    (property "Datasheet" "~" (at 115.57 43.18 0)
+    (property "Footprint" "TerminalBlock_Phoenix:TerminalBlock_Phoenix_MKDS-1,5-4-5.08_1x04_P5.08mm_Horizontal" (at 115.57 40.64 0)
+      (effects (font (size 1.27 1.27)) hide)
+    )
+    (property "Datasheet" "~" (at 115.57 40.64 0)
       (effects (font (size 1.27 1.27)) hide)
     )
@@
     )
   )
-  (symbol (lib_id "Connector:Screw_Terminal_01x04") (at 69.85 40.64 0) (mirror y) (unit 1)
+  (symbol (lib_id "Connector:Screw_Terminal_01x04") (at 69.85 43.18 180) (unit 1)
     (in_bom yes) (on_board yes) (dnp no)
-    (property "Reference" "J2" (at 71.12 31.75 0)
-      (effects (font (size 1.27 1.27)) (justify left))
-    )
-    (property "Value" "CAN Conn" (at 74.93 34.29 0)
-      (effects (font (size 1.27 1.27)) (justify left))
-    )
-    (property "Footprint" "TerminalBlock_Phoenix:TerminalBlock_Phoenix_MKDS-1,5-4-5.08_1x04_P5.08mm_Horizontal" (at 69.85 40.64 0)
-      (effects (font (size 1.27 1.27)) hide)
-    )
-    (property "Datasheet" "~" (at 69.85 40.64 0)
+    (property "Reference" "J2" (at 71.12 52.07 0)
+      (effects (font (size 1.27 1.27)) (justify left))
+    )
+    (property "Value" "CAN Conn" (at 74.93 49.53 0)
+      (effects (font (size 1.27 1.27)) (justify left))
+    )
+    (property "Footprint" "TerminalBlock_Phoenix:TerminalBlock_Phoenix_MKDS-1,5-4-5.08_1x04_P5.08mm_Horizontal" (at 69.85 43.18 0)
+      (effects (font (size 1.27 1.27)) hide)
+    )
+    (property "Datasheet" "~" (at 69.85 43.18 0)
       (effects (font (size 1.27 1.27)) hide)
     )
@@
       (effects (font (size 1.27 1.27)) (justify right))
     )
-    (property "Footprint" "TestPoint:TestPoint_Pad_2.0x2.0mm" (at 60.96 120.65 0)
+    (property "Footprint" "TestPoint:TestPoint_Keystone_5005-5009_Compact" (at 60.96 120.65 0)
       (effects (font (size 1.27 1.27)) hide)
     )
@@
       (effects (font (size 1.27 1.27)))
     )
-    (property "Footprint" "TestPoint:TestPoint_Pad_2.0x2.0mm" (at 208.28 121.92 0)
+    (property "Footprint" "TestPoint:TestPoint_Keystone_5005-5009_Compact" (at 208.28 121.92 0)
       (effects (font (size 1.27 1.27)) hide)
     )
@@
       (effects (font (size 1.27 1.27)) (justify right))
     )
-    (property "Footprint" "TestPoint:TestPoint_Pad_2.0x2.0mm" (at 83.82 154.94 0)
+    (property "Footprint" "TestPoint:TestPoint_Keystone_5005-5009_Compact" (at 83.82 154.94 0)
       (effects (font (size 1.27 1.27)) hide)
     )
@@
       (effects (font (size 1.27 1.27)))
     )
-    (property "Footprint" "TestPoint:TestPoint_Pad_2.0x2.0mm" (at 208.28 132.08 0)
+    (property "Footprint" "TestPoint:TestPoint_Keystone_5005-5009_Compact" (at 208.28 132.08 0)
       (effects (font (size 1.27 1.27)) hide)
     )
@@
       (effects (font (size 1.27 1.27)))
     )
-    (property "Footprint" "TestPoint:TestPoint_Pad_2.0x2.0mm" (at 208.28 142.24 0)
+    (property "Footprint" "TestPoint:TestPoint_Keystone_5005-5009_Compact" (at 208.28 142.24 0)
       (effects (font (size 1.27 1.27)) hide)
     )
@@
       (effects (font (size 1.27 1.27)) (justify right))
     )
-    (property "Footprint" "TestPoint:TestPoint_Pad_2.0x2.0mm" (at 78.74 154.94 0)
+    (property "Footprint" "TestPoint:TestPoint_Keystone_5005-5009_Compact" (at 78.74 154.94 0)
       (effects (font (size 1.27 1.27)) hide)
     )
@@
       (effects (font (size 1.27 1.27)) (justify right))
     )
-    (property "Footprint" "TestPoint:TestPoint_Pad_2.0x2.0mm" (at 74.93 120.65 0)
-      (effects (font (size 1.27 1.27)) hide)
-    )
+    (property "Footprint" "TestPoint:TestPoint_Keystone_5005-5009_Compact" (at 74.93 120.65 0)
+      (effects (font (size 1.27 1.27)) hide)
+    )
