File: design/input_board/input_board.kicad_sch (KiCad schematic)
At the start: 18 parts

Commit message: Finihs schamtic and footprints; DVDD 3.3->2V
Parts:
- removed D2: RED, symbol Device:LED
- removed D5: BLUE, symbol Device:LED
- added D1: BLUE, LED_SMD:LED_1206_3216Metric_Pad1.42x1.75mm_HandSolder, symbol Device:LED
- added D3: RED, LED_SMD:LED_1206_3216Metric_Pad1.42x1.75mm_HandSolder, symbol Device:LED
- D2: renamed from D4; footprint (none) -> LED_SMD:LED_1206_3216Metric_Pad1.42x1.75mm_HandSolder
- D4: renamed from D6; footprint (none) -> LED_SMD:LED_1206_3216Metric_Pad1.42x1.75mm_HandSolder
- H1, H4: footprint (none) -> MountingHole:MountingHole_3.2mm_M3_DIN965_Pad
- H2: renamed from H3; footprint (none) -> MountingHole:MountingHole_3.2mm_M3_DIN965_Pad
- H3: renamed from H2; footprint (none) -> MountingHole:MountingHole_3.2mm_M3_DIN965_Pad
- R1: renamed from R39; footprint (none) -> Resistor_SMD:R_0805_2012Metric_Pad1.20x1.40mm_HandSolder
- R2: renamed from R40; footprint (none) -> Resistor_SMD:R_0805_2012Metric_Pad1.20x1.40mm_HandSolder
- R3: renamed from R41; footprint (none) -> Resistor_SMD:R_0805_2012Metric_Pad1.20x1.40mm_HandSolder
- R4: renamed from R42; footprint (none) -> Resistor_SMD:R_0805_2012Metric_Pad1.20x1.40mm_HandSolder
- TP1, TP6: footprint (none) -> TestPoint:TestPoint_Keystone_5000-5004_Miniature
- TP2: renamed from TP5; footprint (none) -> TestPoint:TestPoint_Keystone_5000-5004_Miniature
- TP3: value 3V3 -> 2V; footprint (none) -> TestPoint:TestPoint_Keystone_5000-5004_Miniature
- TP4: footprint (none) -> TestPoint:TestPoint_Pad_1.5x1.5mm
- TP5: renamed from TP2; footprint (none) -> TestPoint:TestPoint_Keystone_5000-5004_Miniature
Connections:
- net +12V: now also D1.2 (A)
- net at R3.1: now also D3.1 (K)
- net at R1.1: now also D1.1 (K)
- net +3V3 renamed +2V
- net +2V: now also D3.2 (A)
Other:
- sheet 3.3V DVCC renamed 2V DVCC
- sheet 30V AVCC renamed 30V VDDA
- sheet 12V Input ports: added none; removed PGOOD_12V
- sheet 2V DVCC ports: added ISENSE_2V; removed ISENSE_3V3
- sheet 30V VDDA ports: added ISENSE_30V; removed ISENSE_VDDA
- sheet ADC + FVR ports: added CAL; removed none
- sheet MCU ports: added AMP_SEL_0, AMP_SEL_1, AMP_SEL_2, CONVST, FLT_0, FLT_1, FLT_2, FLT_3, IN_SEL_0, IN_SEL_1, IN_SEL_2, IN_SEL_3, IN_SEL_4, IN_SEL_5, ISENSE_12V, ISENSE_2V, ISENSE_30V, MUX_EN, PGOOD_30V, SF_0, SF_1, SF_2, SF_3, SPI1_MISO, SPI1_MOSI, SPI1_SCK, ~{FLT_12V}; removed none
- moved on the sheet: TP5
