File: design/input_board/frontend.kicad_sch (KiCad schematic)
At the start: 26 parts, among them IC1 TMUX7349FPWR, IC2 TMUX7349FPWR, IC3 TMUX7349FPWR, IC4 TMUX7349FPWR, IC5 MUX509IPW, IC6 MUX509IPW, J2 IN1-8, J3 IN 9-18

Commit message: Finihs schamtic and footprints; DVDD 3.3->2V
Parts:
- removed J2: IN1-8, symbol Connector:Screw_Terminal_01x16
- removed J3: IN 9-18, symbol Connector:Screw_Terminal_01x16
- added J3, J4, J5, J6: Screw_Terminal_01x08, TerminalBlock_Phoenix:TerminalBlock_Phoenix_MPT-0,5-8-2.54_1x08_P2.54mm_Horizontal, symbol Connector:Screw_Terminal_01x08
- added J7: Screw_Terminal_01x02, TerminalBlock_Phoenix:TerminalBlock_Phoenix_MPT-0,5-2-2.54_1x02_P2.54mm_Horizontal, symbol Connector:Screw_Terminal_01x02
- C16: renamed from C29; footprint (none) -> Capacitor_SMD:C_0805_2012Metric_Pad1.18x1.45mm_HandSolder
- C17: renamed from C30; footprint (none) -> Capacitor_SMD:C_0805_2012Metric_Pad1.18x1.45mm_HandSolder
- C18: renamed from C27; footprint (none) -> Capacitor_SMD:C_0805_2012Metric_Pad1.18x1.45mm_HandSolder
- C19: renamed from C28; footprint (none) -> Capacitor_SMD:C_0805_2012Metric_Pad1.18x1.45mm_HandSolder
- C20: renamed from C33; footprint (none) -> Capacitor_SMD:C_0805_2012Metric_Pad1.18x1.45mm_HandSolder
- C21: renamed from C34; footprint (none) -> Capacitor_SMD:C_0805_2012Metric_Pad1.18x1.45mm_HandSolder
- C22: renamed from C31; footprint (none) -> Capacitor_SMD:C_0805_2012Metric_Pad1.18x1.45mm_HandSolder
- C23: renamed from C32; footprint (none) -> Capacitor_SMD:C_0805_2012Metric_Pad1.18x1.45mm_HandSolder
- C24: renamed from C35; footprint (none) -> Capacitor_SMD:C_0805_2012Metric_Pad1.18x1.45mm_HandSolder
- C25: renamed from C36; footprint (none) -> Capacitor_SMD:C_0805_2012Metric_Pad1.18x1.45mm_HandSolder
- R23: renamed from R18; footprint (none) -> Resistor_SMD:R_0805_2012Metric_Pad1.20x1.40mm_HandSolder
- R24: renamed from R17; footprint (none) -> Resistor_SMD:R_0805_2012Metric_Pad1.20x1.40mm_HandSolder
- R25: renamed from R21; footprint (none) -> Resistor_SMD:R_0805_2012Metric_Pad1.20x1.40mm_HandSolder
- R26: renamed from R23; footprint (none) -> Resistor_SMD:R_0805_2012Metric_Pad1.20x1.40mm_HandSolder
- R27: renamed from R20; footprint (none) -> Resistor_SMD:R_0805_2012Metric_Pad1.20x1.40mm_HandSolder
- R28: renamed from R19; footprint (none) -> Resistor_SMD:R_0805_2012Metric_Pad1.20x1.40mm_HandSolder
- R29: renamed from R22; footprint (none) -> Resistor_SMD:R_0805_2012Metric_Pad1.20x1.40mm_HandSolder
- R30: renamed from R24; footprint (none) -> Resistor_SMD:R_0805_2012Metric_Pad1.20x1.40mm_HandSolder
- renumbered IC1 to IC2, IC2 to IC4, IC4 to IC5, IC5 to IC7
Connections:
- net GND: now also J7.1 (Pin_1), J7.2 (Pin_2)
- net IN1+: now also J3.1 (Pin_1)
- net IN1-: now also J3.2 (Pin_2)
- net IN10+: now also J5.3 (Pin_3)
- net IN10-: now also J5.4 (Pin_4)
- net IN11+: now also J5.5 (Pin_5)
- net IN11-: now also J5.6 (Pin_6)
- net IN12+: now also J5.7 (Pin_7)
- net IN12-: now also J5.8 (Pin_8)
- net IN13+: now also J6.1 (Pin_1)
- net IN13-: now also J6.2 (Pin_2)
- net IN14+: now also J6.3 (Pin_3)
- net IN14-: now also J6.4 (Pin_4)
- net IN15+: now also J6.5 (Pin_5)
- net IN15-: now also J6.6 (Pin_6)
- net IN16+: now also J6.7 (Pin_7)
- net IN16-: now also J6.8 (Pin_8)
- net IN2+: now also J3.3 (Pin_3)
- net IN2-: now also J3.4 (Pin_4)
- net IN3+: now also J3.5 (Pin_5)
- net IN3-: now also J3.6 (Pin_6)
- net IN4+: now also J3.7 (Pin_7)
- net IN4-: now also J3.8 (Pin_8)
- net IN5+: now also J4.1 (Pin_1)
- net IN5-: now also J4.2 (Pin_2)
- net IN6+: now also J4.3 (Pin_3)
- net IN6-: now also J4.4 (Pin_4)
- net IN7+: now also J4.5 (Pin_5)
- net IN7-: now also J4.6 (Pin_6)
- net IN8+: now also J4.7 (Pin_7)
- net IN8-: now also J4.8 (Pin_8)
- net IN9+: now also J5.1 (Pin_1)
- net IN9-: now also J5.2 (Pin_2)
- net +3V3 renamed +2V

Commit message: Layout v1, its bad
Parts:
- added J11: Screw_Terminal_01x02, TerminalBlock_Phoenix:TerminalBlock_Phoenix_MPT-0,5-2-2.54_1x02_P2.54mm_Horizontal, symbol Connector:Screw_Terminal_01x02
Connections:
- net GND: now also J11.1 (Pin_1), J11.2 (Pin_2)
Changed lines of the file:
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@@
 	)
 	(junction
+		(at 54.61 186.69)
+		(diameter 0)
+		(color 0 0 0 0)
+	)
+	(junction
 		(at 252.73 55.88)
 		(diameter 0)
@@
 	(wire
 		(pts
+			(xy 58.42 186.69) (xy 58.42 190.5)
+		)
+		(stroke
+			(width 0)
+			(type default)
+		)
+	)
+	(wire
+		(pts
 			(xy 140.97 102.87) (xy 140.97 87.63)
 		)
@@
 	(wire
 		(pts
+			(xy 53.34 189.23) (xy 54.61 189.23)
+		)
+		(stroke
+			(width 0)
+			(type default)
+		)
+	)
+	(wire
+		(pts
 			(xy 151.13 55.88) (xy 148.59 55.88)
 		)
@@
 	(wire
 		(pts
+			(xy 54.61 186.69) (xy 54.61 189.23)
+		)
+		(stroke
+			(width 0)
+			(type default)
+		)
+	)
+	(wire
+		(pts
 			(xy 130.81 138.43) (xy 144.78 138.43)
 		)
@@
 	(wire
 		(pts
+			(xy 54.61 186.69) (xy 58.42 186.69)
+		)
+		(stroke
+			(width 0)
+			(type default)
+		)
+	)
+	(wire
+		(pts
 			(xy 262.89 21.59) (xy 269.24 21.59)
 		)
@@
 	(wire
 		(pts
+			(xy 53.34 186.69) (xy 54.61 186.69)
+		)
+		(stroke
+			(width 0)
+			(type default)
+		)
+	)
+	(wire
+		(pts
 			(xy 158.75 139.7) (xy 158.75 140.97)
 		)
@@
 	)
 	(symbol
+		(lib_id "Connector:Screw_Terminal_01x02")
+		(at 48.26 189.23 180)
+		(unit 1)
+		(exclude_from_sim no)
+		(in_bom yes)
+		(on_board yes)
+		(dnp no)
+		(property "Reference" "J11"
+			(at 33.02 185.42 0)
+			(effects
+				(font
+					(size 1.27 1.27)
+				)
+			)
+		)
+		(property "Value" "Screw_Terminal_01x02"
+			(at 33.02 187.96 0)
+			(effects
+				(font
+					(size 1.27 1.27)
+				)
+			)
+		)
+		(property "Footprint" "TerminalBlock_Phoenix:TerminalBlock_Phoenix_MPT-0,5-2-2.54_1x02_P2.54mm_Horizontal"
+			(at 48.26 189.23 0)
+			(effects
+				(font
+					(size 1.27 1.27)
+				)
+				(hide yes)
+			)
+		)
+		(property "Datasheet" "~"
+			(at 48.26 189.23 0)
+			(effects
+				(font
+					(size 1.27 1.27)
+				)
+				(hide yes)
+			)
+		)
+		(property "Description" "Generic screw terminal, single row, 01x02, script generated (kicad-library-utils/schlib/autogen/connector/)"
+			(at 48.26 189.23 0)
+			(effects
+				(font
+					(size 1.27 1.27)
+				)
+				(hide yes)
+			)
+		)
+		(pin "2"
+		)
+		(pin "1"
+		)
+		(instances
+			(project "input_board"
+				(path "/edc2dfd5-6e83-475f-94b9-1e03bbedf967/7f9a9c17-cbc2-43ce-8edf-083c96183002"
+					(reference "J11")
+					(unit 1)
+				)
+			)
+		)
+	)
+	(symbol
 		(lib_id "input_board:+2V")
 		(at 191.77 45.72 0)
@@
 					(unit 1)
 				)
+			)
+		)
+	)
+	(symbol
+		(lib_id "power:GND")
+		(at 58.42 190.5 0)
+		(unit 1)
+		(exclude_from_sim no)
+		(in_bom yes)
+		(on_board yes)
+		(dnp no)
+		(fields_autoplaced yes)
+		(property "Reference" "#PWR0143"
+			(at 58.42 196.85 0)
+			(effects
+				(font
+					(size 1.27 1.27)
+				)
+				(hide yes)
+			)
+		)
+		(property "Value" "GND"
+			(at 58.42 195.58 0)
+			(effects
+				(font
+					(size 1.27 1.27)
+				)
+			)
+		)
+		(property "Footprint" ""
+			(at 58.42 190.5 0)
+			(effects
+				(font
+					(size 1.27 1.27)
+				)
+				(hide yes)
+			)
+		)
+		(property "Datasheet" ""
+			(at 58.42 190.5 0)
+			(effects
+				(font
+					(size 1.27 1.27)
+				)
+				(hide yes)
+			)
+		)
+		(property "Description" "Power symbol creates a global label with name \"GND\" , ground"
+			(at 58.42 190.5 0)
+			(effects
+				(font
+					(size 1.27 1.27)
+				)
+				(hide yes)
+			)
+		)
+		(pin "1"
+		)
+		(instances
+			(project "input_board"
+				(path "/edc2dfd5-6e83-475f-94b9-1e03bbedf967/7f9a9c17-cbc2-43ce-8edf-083c96183002"
+					(reference "#PWR0143")
+					(unit 1)
+				)
