File: design/input_board/input_board.kicad_pcb (KiCad board)
At the start: 6 copper layers, 111.8 x 61 mm, 179 parts, among them IC1 LM5157RTER, IC10 ADS8860IDGSR, IC2 TMUX7349FPWR, IC3 TMUX7349FPWR, IC4 TMUX7349FPWR, IC5 TMUX7349FPWR, IC6 MUX509IPW, IC7 MUX509IPW, IC8 MUX36D08IPW, IC9 MUX508IPW, J1 Screw_Terminal_01x02, J10 Programmer, J11 Screw_Terminal_01x02, J2 Screw_Terminal_01x03, J3 Screw_Terminal_01x08, J4 Screw_Terminal_01x08, J5 Screw_Terminal_01x08, J6 Screw_Terminal_01x08, J7 Screw_Terminal_01x02, J8 USB_B, J9 CAN, Q1 CSD19537Q3, Q2 BSS138, U1 TPS26631PWP, U10 INA849DGK, U11 INA849DGK, U12 REF6050xDGK, U13 uA7805, U14 TPS76933, U15 MCP2562, U16 STM32H750ZBTx, U17 TPS565201, U18 INA180A3, U2 TPS7A4701xRGW, U3 INA290A3, U4 INA849DGK, U5 INA849DGK, U6 INA849DGK, U7 INA849DGK, U8 INA849DGK, U9 INA849DGK

Commit message: Prod files, update input #s
Other:
- board text added: "IN10+"
- board text added: "IN10-"
- board text added: "IN11+"
- board text added: "IN11-"
- board text added: "IN12+"
- board text added: "IN12-"
- board text added: "IN13+"
- board text added: "IN13-"
- board text added: "IN14+"
- board text added: "IN14-"
- board text added: "IN15+"
- board text added: "IN15-"
- board text added: "IN16+"
- board text added: "IN16-"
- board text added: "IN2+"
- board text added: "IN2-"
- board text added: "IN3+"
- board text added: "IN3-"
- board text added: "IN4+"
- board text added: "IN4-"
- board text added: "IN5+"
- board text added: "IN5-"
- board text added: "IN6+"
- board text added: "IN6-"
- board text added: "IN7+"
- board text added: "IN7-"
- board text added: "IN8+"
- board text added: "IN8-"
- board text added: "IN9+"
- board text added: "IN9-"
