File: design/DAQ Patch Panel/sensor_comp.kicad_sch (KiCad schematic)
At the start: 13 parts

Commit message: Footprint and Hierarchal Sheets
Footprint for 6 screw terminal block added and sensor components made into hierarchical sheets
Changed lines of the file:
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@@
     (effects (font (size 1.27 1.27)) (justify left bottom))
   )
-  (label "IN 1" (at 105.41 90.17 90) (fields_autoplaced)
-    (effects (font (size 1.27 1.27)) (justify left bottom))
+  (label "IN 1" (at 105.41 90.17 180) (fields_autoplaced)
+    (effects (font (size 1.27 1.27)) (justify right bottom))
   )
   (label "IN 1" (at 165.1 93.98 180) (fields_autoplaced)
@@
     (effects (font (size 1.27 1.27)) (justify right bottom))
   )
-  (label "IN 2" (at 140.97 91.44 90) (fields_autoplaced)
-    (effects (font (size 1.27 1.27)) (justify left bottom))
+  (label "IN 2" (at 140.97 91.44 180) (fields_autoplaced)
+    (effects (font (size 1.27 1.27)) (justify right bottom))
   )
   (label "POWER" (at 144.78 76.2 0) (fields_autoplaced)
@@
   )
   (symbol (lib_id "power:GND") (at 147.32 114.3 0) (unit 1)
-    (in_bom yes) (on_board yes) (dnp no) (fields_autoplaced)
+    (in_bom yes) (on_board yes) (dnp no)
     (property "Reference" "#PWR01" (at 147.32 120.65 0)
       (effects (font (size 1.27 1.27)) hide)
     )
-    (property "Value" "GND" (at 147.32 118.11 90)
+    (property "Value" "GND" (at 135.89 119.38 0)
       (effects (font (size 1.27 1.27)) (justify right))
     )
@@
   (symbol (lib_name "Jumper_3_Open_1") (lib_id "Jumper:Jumper_3_Open") (at 140.97 95.25 180) (unit 1)
     (in_bom yes) (on_board yes) (dnp no)
-    (property "Reference" "JP2" (at 140.97 97.79 90)
-      (effects (font (size 1.27 1.27)) (justify left))
-    )
-    (property "Value" "RESISTOR JUMPER 1" (at 138.43 97.79 90)
+    (property "Reference" "JP2" (at 142.24 87.63 0)
+      (effects (font (size 1.27 1.27)) (justify left))
+    )
+    (property "Value" "RESISTOR JUMPER 1" (at 149.86 85.09 0)
       (effects (font (size 1.27 1.27)) (justify left))
     )
@@
   (symbol (lib_id "Device:R_US") (at 99.06 105.41 0) (unit 1)
     (in_bom yes) (on_board yes) (dnp no)
-    (property "Reference" "R6" (at 96.52 105.41 90)
-      (effects (font (size 1.27 1.27)))
-    )
-    (property "Value" "100R 1%" (at 93.98 106.68 90)
+    (property "Reference" "R6" (at 116.84 104.14 0)
+      (effects (font (size 1.27 1.27)))
+    )
+    (property "Value" "100R 1%" (at 118.11 106.68 0)
       (effects (font (size 1.27 1.27)))
     )
@@
   (symbol (lib_id "Device:R_US") (at 111.76 105.41 0) (unit 1)
     (in_bom yes) (on_board yes) (dnp no)
-    (property "Reference" "R5" (at 114.3 105.41 90)
-      (effects (font (size 1.27 1.27)))
-    )
-    (property "Value" "10k 1%" (at 116.84 105.41 90)
+    (property "Reference" "R5" (at 95.25 104.14 0)
+      (effects (font (size 1.27 1.27)))
+    )
+    (property "Value" "10k 1%" (at 93.98 106.68 0)
       (effects (font (size 1.27 1.27)))
     )
@@
   (symbol (lib_id "Device:R_US") (at 134.62 106.68 0) (unit 1)
     (in_bom yes) (on_board yes) (dnp no)
-    (property "Reference" "R2" (at 132.08 106.68 90)
-      (effects (font (size 1.27 1.27)))
-    )
-    (property "Value" "100R 1%" (at 129.54 106.68 90)
+    (property "Reference" "R2" (at 130.81 106.68 0)
+      (effects (font (size 1.27 1.27)))
+    )
+    (property "Value" "100R 1%" (at 129.54 104.14 0)
       (effects (font (size 1.27 1.27)))
     )
@@
       (effects (font (size 1.27 1.27)) hide)
     )
-    (property "Value" "GND" (at 96.52 113.03 90)
+    (property "Value" "GND" (at 101.6 118.11 0)
       (effects (font (size 1.27 1.27)) (justify right))
     )
@@
   (symbol (lib_name "Jumper_3_Open_1") (lib_id "Jumper:Jumper_3_Open") (at 105.41 93.98 180) (unit 1)
     (in_bom yes) (on_board yes) (dnp no)
-    (property "Reference" "JP7" (at 105.41 96.52 90)
-      (effects (font (size 1.27 1.27)) (justify left))
-    )
-    (property "Value" "RESISTOR JUMPER 2" (at 102.87 96.52 90)
+    (property "Reference" "JP7" (at 106.68 86.36 0)
+      (effects (font (size 1.27 1.27)) (justify left))
+    )
+    (property "Value" "RESISTOR JUMPER 2" (at 114.3 83.82 0)
       (effects (font (size 1.27 1.27)) (justify left))
     )
@@
   )
   (symbol (lib_id "power:GND") (at 111.76 113.03 0) (unit 1)
-    (in_bom yes) (on_board yes) (dnp no) (fields_autoplaced)
+    (in_bom yes) (on_board yes) (dnp no)
     (property "Reference" "#PWR08" (at 111.76 119.38 0)
       (effects (font (size 1.27 1.27)) hide)
     )
-    (property "Value" "GND" (at 111.76 116.84 90)
+    (property "Value" "GND" (at 114.3 118.11 0)
       (effects (font (size 1.27 1.27)) (justify right))
     )
@@
       (effects (font (size 1.27 1.27)) hide)
     )
-    (property "Value" "GND" (at 133.35 118.11 90)
+    (property "Value" "GND" (at 149.86 119.38 0)
       (effects (font (size 1.27 1.27)) (justify right))
     )

Commit message: Files Renamed and Changes Implemented
Renamed project to Daq Patch Panel
Updated 4 way jumper footprints
Renamed input screw terminal
Parts:
- JP1: footprint Library:4-Pole Jumper -> Library:4-Way-Jumper
Changed lines of the file:
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@@
     (pin "1")
     (instances
-      (project "DAQ_Power_Patch"
+      (project "DAQ_Patch_Panel"
         (path "/da75d2ac-4c40-407d-8f74-3497a5ffc88d"
           (reference "#PWR01") (unit 1)
@@
     (pin "3")
     (instances
-      (project "DAQ_Power_Patch"
+      (project "DAQ_Patch_Panel"
         (path "/da75d2ac-4c40-407d-8f74-3497a5ffc88d"
           (reference "JP2") (unit 1)
@@
     (pin "2")
     (instances
-      (project "DAQ_Power_Patch"
+      (project "DAQ_Patch_Panel"
         (path "/da75d2ac-4c40-407d-8f74-3497a5ffc88d"
           (reference "F1") (unit 1)
@@
     (pin "2")
     (instances
-      (project "DAQ_Power_Patch"
+      (project "DAQ_Patch_Panel"
         (path "/da75d2ac-4c40-407d-8f74-3497a5ffc88d"
           (reference "R6") (unit 1)
@@
     (pin "1")
     (instances
-      (project "DAQ_Power_Patch"
+      (project "DAQ_Patch_Panel"
         (path "/da75d2ac-4c40-407d-8f74-3497a5ffc88d"
           (reference "#PWR06") (unit 1)
@@
     (pin "1")
     (instances
-      (project "DAQ_Power_Patch"
+      (project "DAQ_Patch_Panel"
         (path "/da75d2ac-4c40-407d-8f74-3497a5ffc88d"
           (reference "#PWR05") (unit 1)
@@
     (pin "2")
     (instances
-      (project "DAQ_Power_Patch"
+      (project "DAQ_Patch_Panel"
         (path "/da75d2ac-4c40-407d-8f74-3497a5ffc88d"
           (reference "R4") (unit 1)
@@
     (pin "2")
     (instances
-      (project "DAQ_Power_Patch"
+      (project "DAQ_Patch_Panel"
         (path "/da75d2ac-4c40-407d-8f74-3497a5ffc88d"
           (reference "C1") (unit 1)
@@
     (pin "1")
     (instances
-      (project "DAQ_Power_Patch"
+      (project "DAQ_Patch_Panel"
         (path "/da75d2ac-4c40-407d-8f74-3497a5ffc88d"
           (reference "#PWR018") (unit 1)
@@
     (pin "1")
     (instances
-      (project "DAQ_Power_Patch"
+      (project "DAQ_Patch_Panel"
         (path "/da75d2ac-4c40-407d-8f74-3497a5ffc88d"
           (reference "#PWR07") (unit 1)
@@
     (pin "2")
     (instances
-      (project "DAQ_Power_Patch"
+      (project "DAQ_Patch_Panel"
         (path "/da75d2ac-4c40-407d-8f74-3497a5ffc88d"
           (reference "C2") (unit 1)
@@
     (pin "1")
     (instances
-      (project "DAQ_Power_Patch"
+      (project "DAQ_Patch_Panel"
         (path "/da75d2ac-4c40-407d-8f74-3497a5ffc88d"
           (reference "#PWR03") (unit 1)
@@
     (pin "2")
     (instances
-      (project "DAQ_Power_Patch"
+      (project "DAQ_Patch_Panel"
         (path "/da75d2ac-4c40-407d-8f74-3497a5ffc88d"
           (reference "R5") (unit 1)
@@
     (pin "2")
     (instances
-      (project "DAQ_Power_Patch"
+      (project "DAQ_Patch_Panel"
         (path "/da75d2ac-4c40-407d-8f74-3497a5ffc88d"
           (reference "R3") (unit 1)
@@
     (pin "2")
     (instances
-      (project "DAQ_Power_Patch"
+      (project "DAQ_Patch_Panel"
         (path "/da75d2ac-4c40-407d-8f74-3497a5ffc88d"
           (reference "R2") (unit 1)
@@
     (pin "1")
     (instances
-      (project "DAQ_Power_Patch"
+      (project "DAQ_Patch_Panel"
         (path "/da75d2ac-4c40-407d-8f74-3497a5ffc88d"
           (reference "#PWR04") (unit 1)
@@
     (pin "1")
     (instances
-      (project "DAQ_Power_Patch"
+      (project "DAQ_Patch_Panel"
         (path "/da75d2ac-4c40-407d-8f74-3497a5ffc88d"
           (reference "#PWR09") (unit 1)
@@
     (pin "2")
     (instances
-      (project "DAQ_Power_Patch"
+      (project "DAQ_Patch_Panel"
         (path "/da75d2ac-4c40-407d-8f74-3497a5ffc88d"
           (reference "R1") (unit 1)
@@
     (pin "3")
     (instances
-      (project "DAQ_Power_Patch"
+      (project "DAQ_Patch_Panel"
         (path "/da75d2ac-4c40-407d-8f74-3497a5ffc88d"
           (reference "JP7") (unit 1)
@@
       (effects (font (size 1.27 1.27)))
     )
-    (property "Footprint" "Library:4-Pole Jumper" (at 116.84 62.23 0)
+    (property "Footprint" "Library:4-Way-Jumper" (at 116.84 62.23 0)
       (effects (font (size 1.27 1.27)) hide)
     )
@@
     (pin "5")
     (instances
-      (project "DAQ_Power_Patch"
+      (project "DAQ_Patch_Panel"
         (path "/da75d2ac-4c40-407d-8f74-3497a5ffc88d"
           (reference "JP1") (unit 1)
@@
     (pin "1")
     (instances
-      (project "DAQ_Power_Patch"
+      (project "DAQ_Patch_Panel"
         (path "/da75d2ac-4c40-407d-8f74-3497a5ffc88d"
           (reference "#PWR016") (unit 1)
@@
     (pin "1")
     (instances
-      (project "DAQ_Power_Patch"
+      (project "DAQ_Patch_Panel"
         (path "/da75d2ac-4c40-407d-8f74-3497a5ffc88d"
           (reference "#PWR08") (unit 1)
@@
     (pin "1")
     (instances
-      (project "DAQ_Power_Patch"
+      (project "DAQ_Patch_Panel"
         (path "/da75d2ac-4c40-407d-8f74-3497a5ffc88d"
           (reference "#PWR02") (unit 1)
@@
     (pin "3")
     (instances
-      (project "DAQ_Power_Patch"
+      (project "DAQ_Patch_Panel"
         (path "/da75d2ac-4c40-407d-8f74-3497a5ffc88d"
           (reference "JP4") (unit 1)

Commit message: Latest Review Changes
Parts:
- removed JP7: RESISTOR JUMPER 2, Connector_PinHeader_2.54mm:PinHeader_1x03_P2.54mm_Vertical, symbol Jumper:Jumper_3_Open
- removed R5: 10k 1%, Resistor_SMD:R_0805_2012Metric_Pad1.20x1.40mm_HandSolder, symbol Device:R_US
- removed R6: 100R 1%, Resistor_SMD:R_0805_2012Metric_Pad1.20x1.40mm_HandSolder, symbol Device:R_US
- added JP2: RESISTOR JUMPER 2, Connector_PinHeader_2.54mm:PinHeader_1x03_P2.54mm_Vertical, symbol Jumper:Jumper_3_Open
- added R1: 10k 1%, Resistor_SMD:R_0805_2012Metric_Pad1.20x1.40mm_HandSolder, symbol Device:R_US
- added R2: 100R 1%, Resistor_SMD:R_0805_2012Metric_Pad1.20x1.40mm_HandSolder, symbol Device:R_US
Connections:
- net +10V: now also JP1.4 (C); no longer JP1.5 (C)
- net +20V: now also JP1.5 (C); no longer JP1.4 (C)
- net GND: now also R1.2, R2.2
- net IN1: now also JP2.2 (C)
- new net: JP2.3 (B), R2.1
- new net: JP2.1 (A), R1.1
Other:
- moved on the sheet: R1, R2, R3

Commit message: Jack's Nitpicks Fixing
Changed lines of the file:
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@@
       (effects (font (size 1.27 1.27)) hide)
     )
-    (property "Value" "GND" (at 149.86 119.38 0)
-      (effects (font (size 1.27 1.27)) (justify right))
+    (property "Value" "GND" (at 148.59 119.38 0)
+      (effects (font (size 1.27 1.27)))
     )
     (property "Footprint" "" (at 148.59 114.3 0)
@@
       (effects (font (size 1.27 1.27)) hide)
     )
-    (property "Value" "GND" (at 111.76 119.38 0)
-      (effects (font (size 1.27 1.27)) (justify right))
+    (property "Value" "GND" (at 110.49 119.38 0)
+      (effects (font (size 1.27 1.27)))
     )
     (property "Footprint" "" (at 110.49 114.3 0)
@@
       (effects (font (size 1.27 1.27)) hide)
     )
-    (property "Value" "GND" (at 96.52 119.38 0)
-      (effects (font (size 1.27 1.27)) (justify right))
+    (property "Value" "GND" (at 95.25 119.38 0)
+      (effects (font (size 1.27 1.27)))
     )
     (property "Footprint" "" (at 95.25 114.3 0)
@@
   )
   (symbol (lib_id "power:GND") (at 184.15 102.87 0) (unit 1)
-    (in_bom yes) (on_board yes) (dnp no) (fields_autoplaced)
+    (in_bom yes) (on_board yes) (dnp no)
     (property "Reference" "#PWR018" (at 184.15 109.22 0)
       (effects (font (size 1.27 1.27)) hide)
     )
-    (property "Value" "GND" (at 186.69 104.14 0)
-      (effects (font (size 1.27 1.27)) (justify left))
+    (property "Value" "GND" (at 184.15 107.95 0)
+      (effects (font (size 1.27 1.27)))
     )
     (property "Footprint" "" (at 184.15 102.87 0)
@@
   (symbol (lib_id "Device:R_US") (at 95.25 106.68 0) (mirror y) (unit 1)
     (in_bom yes) (on_board yes) (dnp no)
-    (property "Reference" "R2" (at 100.33 107.95 0)
-      (effects (font (size 1.27 1.27)))
-    )
-    (property "Value" "100R 1%" (at 101.6 105.41 0)
+    (property "Reference" "R2" (at 100.33 105.41 0)
+      (effects (font (size 1.27 1.27)))
+    )
+    (property "Value" "100R 1%" (at 101.6 107.95 0)
       (effects (font (size 1.27 1.27)))
     )
@@
   (symbol (lib_id "Device:R_US") (at 110.49 106.68 0) (mirror y) (unit 1)
     (in_bom yes) (on_board yes) (dnp no)
-    (property "Reference" "R1" (at 105.41 106.68 90)
-      (effects (font (size 1.27 1.27)))
-    )
-    (property "Value" "10k 1%" (at 107.95 106.68 90)
+    (property "Reference" "R1" (at 114.3 105.41 0)
+      (effects (font (size 1.27 1.27)))
+    )
+    (property "Value" "10k 1%" (at 115.57 107.95 0)
       (effects (font (size 1.27 1.27)))
     )
@@
   (symbol (lib_id "Device:R_US") (at 133.35 106.68 0) (unit 1)
     (in_bom yes) (on_board yes) (dnp no)
-    (property "Reference" "R2" (at 129.54 106.68 0)
-      (effects (font (size 1.27 1.27)))
-    )
-    (property "Value" "100R 1%" (at 128.27 104.14 0)
+    (property "Reference" "R2" (at 137.16 105.41 0)
+      (effects (font (size 1.27 1.27)))
+    )
+    (property "Value" "100R 1%" (at 139.7 107.95 0)
       (effects (font (size 1.27 1.27)))
     )
@@
   (symbol (lib_id "Device:R_US") (at 148.59 106.68 0) (unit 1)
     (in_bom yes) (on_board yes) (dnp no)
-    (property "Reference" "R1" (at 153.67 106.68 90)
-      (effects (font (size 1.27 1.27)))
-    )
-    (property "Value" "10k 1%" (at 151.13 106.68 90)
+    (property "Reference" "R1" (at 153.67 105.41 0)
+      (effects (font (size 1.27 1.27)))
+    )
+    (property "Value" "10k 1%" (at 153.67 107.95 0)
       (effects (font (size 1.27 1.27)))
     )
@@
   )
   (symbol (lib_id "power:GND") (at 182.88 128.27 0) (unit 1)
-    (in_bom yes) (on_board yes) (dnp no) (fields_autoplaced)
+    (in_bom yes) (on_board yes) (dnp no)
     (property "Reference" "#PWR016" (at 182.88 134.62 0)
       (effects (font (size 1.27 1.27)) hide)
     )
-    (property "Value" "GND" (at 185.42 129.54 0)
-      (effects (font (size 1.27 1.27)) (justify left))
+    (property "Value" "GND" (at 182.88 133.35 0)
+      (effects (font (size 1.27 1.27)))
     )
     (property "Footprint" "" (at 182.88 128.27 0)
@@
       (effects (font (size 1.27 1.27)) hide)
     )
-    (property "Value" "GND" (at 134.62 119.38 0)
-      (effects (font (size 1.27 1.27)) (justify right))
+    (property "Value" "GND" (at 133.35 119.38 0)
+      (effects (font (size 1.27 1.27)))
     )
     (property "Footprint" "" (at 133.35 114.3 0)

Commit message: First draft PCB
Parts:
- F2: renamed from F1; value 50mA -> 50mA
- renumbered C1 to C3, C2 to C4, JP4 to JP5, JP2 to JP6, JP1 to JP7, JP2 to JP8, R2 to R1, R1 to R10, R3 to R11, R4 to R12, R1 to R2, R2 to R9
Connections:
- net +20V renamed +24V
